File: sheets/connectors.kicad_sch (KiCad schematic)
At the start: 0 parts

Commit message: Schematic capture: MCU and NVM (p4), connectors (p9); ERC clean
Page 4: S32K344 in eight boxed units. The supply unit has decoupling per
NXP HDG Rev E2 Table 2; each port unit shows its pin plan and firmware
notes (D-14 as adopted). Pins were checked against NXP's IOMUX table:
EMAC RMII per NXP's TJA1100 use case, LPSPI4 switch chain, LPSPI2 log
flash, LPI2C0 telemetry, ADC1/ADC2 inputs, EIRQ fault lines, SWD and an
LPUART0 debug port. Also the IS25LP032D flash, the Cortex 10-pin header
and the I2C pull-ups.

Page 9: placeholder battery, return, T1S and MX150 output connectors
(all TBD selections), mirrored with pin 1 at the top (D-43), and the
PWR_FLAGs for nets entering the board.

ERC: 0 violations. 17 items are excluded in node60.kicad_pro, each with
its reason (D-52): parallel output pins typed power output in the
library (to be retyped there), and two LAN8670 pins tied to VSS per the
datasheet.

Co-Authored-By: Claude Opus 5.5 <noreply@anthropic.com>
Parts:
- added J: Battery input (TBD), symbol Connector_Generic:Conn_01x01
- added J: T1S 2-way (TBD), symbol Connector_Generic:Conn_01x02
- added J: Power return (TBD), symbol Connector_Generic:Conn_01x01
- added J: MX150 outputs (TBD), symbol Connector_Generic:Conn_01x06
Connections:
- new net GND: J.1 (Pin_1)
- new net OUT1: J.1 (Pin_1)
- new net OUT2: J.2 (Pin_2)
- new net OUT3: J.3 (Pin_3)
- new net OUT4: J.4 (Pin_4)
- new net OUT5: J.5 (Pin_5)
- new net OUT6: J.6 (Pin_6)
- new net T1S_N: J.2 (Pin_2)
- new net T1S_P: J.1 (Pin_1)
- new net VBAT_IN: J.1 (Pin_1)
Other:
- note added: "10BASE-T1S pair, sealed 2-way (J903)"
- note added: "Battery input, 60 A (J901)"
- note added: "CONNECTORS (Node60 harness page; REQ-NET-001: exactly four node conductors: T1S pair, battery, ground) All connector parts are PLACEHOLDERS (generic symbols) until the mating sets are selected and frozen together: housings, terminals, seals, wire sizes and keys (harness page, connector freeze condition). J901 battery input: Metri-Pack 480/630 class, or a dual feed with each feed fused; prove the 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"
- note added: "Outputs 1-6, MX150 sealed, 10 A each (J904)"
- note added: "Power flags (ERC)"
- note added: "Power return, 60 A (J902)"
- title: Node60 -> Node60 · K · Connectors (p9)
