File: sheets/regulators.kicad_sch (KiCad schematic)
At the start: 40 parts

Commit message: Swap placeholders for merged DropOut library parts
Library bumped to ce98ecf (PRs #15, #16, #18, #19, #20, #21 merged).
Now real parts: IAUTN08S5N012LATMA1 (Q201-Q204, dual gate: G_ON and
G_LIN both driven), CSS2725FTL250 (R201, 2-terminal: sense nets are
VBAT_D / VBAT_Q2D with Kelvin taps from the pads in layout),
TPS7B8133QWDRVRQ1 (U301, COUT 2.2uF per its 1-200 uF requirement),
NCU18XH103F6SRB (RT201, RT601-801), Wurth 74438356022HT / 74438356010HT
buck inductors and Harwin S1751-46R GND loops (user's picks 2026-10-23),
1 mm pad test points and DT13-2P output headers. The library pin-type
fixes cut the ERC exclusions from 17 to 2. parts.yaml records the
library symbols; the library tables list the new libraries.

Co-Authored-By: Claude Opus 5.5 <noreply@anthropic.com>
Parts:
- C: value 1uF -> 2.2uF; Package 0402 -> 0603; Voltage 16V -> 10V
- L: value 2.2uH -> 74438356022HT; footprint (none) -> DropOut_Inductor_SMD:L_Wuerth_MAPI-4020; symbol Device:L -> DropOut_Inductor:74438356022HT; DigiKey_PN (none) -> 732-74438356022HTCT-ND; MPN (none) -> 74438356022HT; Manufacturer (none) -> Würth Elektronik; Mouser_PN (none) -> 710-74438356022HT; Placeholder PLACEHOLDER: awaiting DropOut_Inductor buck inductor (libra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 -> (none); Temperature_Grade (none) -> AEC-Q200 Grade 0, -55 to +150 °C operating (-55 to +110 °C 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
- L: value 1uH -> 74438356010HT; footprint (none) -> DropOut_Inductor_SMD:L_Wuerth_MAPI-4020; symbol Device:L -> DropOut_Inductor:74438356010HT; DigiKey_PN (none) -> 732-74438356010HTCT-ND; MPN (none) -> 74438356010HT; Manufacturer (none) -> Würth Elektronik; Mouser_PN (none) -> 710-74438356010HT; Placeholder PLACEHOLDER: awaiting DropOut_Inductor buck inductor (libra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 -> (none); Temperature_Grade (none) -> AEC-Q200 Grade 0, -55 to +150 °C operating (-55 to +110 °C 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
- U: value LDO -> TPS7B8133QWDRVRQ1; footprint (none) -> DropOut_Package_DFN_QFN:Texas_DRV0006A_WSON-6-1EP_2x2mm_P0.65mm_EP1x1.6mm; symbol Connector_Generic:Conn_01x04 -> DropOut_Power:TPS7B8133QWDRVRQ1; DigiKey_PN (none) -> 296-TPS7B8133QWDRVRQ1CT-ND; MPN (none) -> TPS7B8133QWDRVRQ1; Manufacturer (none) -> Texas Instruments; Mouser_PN (none) -> 595-PS7B8133QWDRVRQ1; Placeholder PLACEHOLDER: TBD part: selection pending user decision (fin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 -> (none); Temperature_Grade (none) -> AEC-Q100 Grade 1, TJ -40 to +150 °C
Connections:
- net GND: now also U.3 (GND), U.7 (EP)
- net VDDAU_AON_REG: now also U.6 (OUT); no longer U.3 (Pin_3)
- no-connect marks 14 -> 15
Other:
- note added: "Always-on LAN8670 VDDAU supply: TPS7B8133-Q1 nanopower LDO (U301)"
- note removed: "Always-on LAN8670 VDDAU supply: nanopower LDO, PLACEHOLDER (U301)"
- moved on the sheet: C, R

Commit message: Swap all resistors, capacitors and test points for DropOut parts
Library bumped to 752b63c (PR #22: 83 AEC-Q200 chip resistors and MLCCs,
PR #24: passive symbol layout). Each passive is now a real part, chosen
by rule: exact value and dielectric, tolerance and voltage at least as
good, the drawn package else the next larger, then manufacturer order;
the other built sources stay in the library as alternates.

Where the library has no part in the drawn package: 10nF C0G, 4.7nF C0G,
1uF 16V and 470nF 16V 0402 -> 0603; 68nF C0G, 100nF C0G and 10uF 16V
0805 -> 1206; 32k 1% -> 0.1% (TNPW060332K0BEEA); CCAP 1uF 50V (not built)
-> 1uF 100V 1206. 0R debug links on regulator outputs use the 5 A
CRCW06030000Z0EAHP jumper.

Also fixes test points: f9af1d2 described them as swapped, but they were
still stock symbols. They are now TestPoint_Pad_D1.0mm (signals) and
Harwin S1751-46R (GND loops).

Only placeholders left: L201 / C208 (EMI filter, TBD) and J901-J903.

Co-Authored-By: Claude Opus 5.5 <noreply@anthropic.com>
Parts:
- C: footprint (none) -> DropOut_Capacitor_SMD:C_1210_3225Metric; symbol Device:C -> DropOut_Capacitor:CNA6P1X7R2A475K250AE; Case (none) -> 1210; DigiKey_PN (none) -> 445-181409-1-ND; MPN (none) -> CNA6P1X7R2A475K250AE; Manufacturer (none) -> TDK; Mouser_PN (none) -> 810-CNA6P1X7R2A475K2; Notes (none) -> TDK makes this value only in its CNA soft termination serie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; Package 1210 -> (none); Placeholder PLACEHOLDER: awaiting DropOut_Resistor/DropOut_Capacitor pa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 -> (none); Temperature_Grade (none) -> AEC-Q200, -55 to +125 °C; Tolerance 10% -> ±10%
- C: footprint (none) -> DropOut_Capacitor_SMD:C_0603_1608Metric; symbol Device:C -> DropOut_Capacitor:AC0603KRX7R6BB225; Case (none) -> 0603; DigiKey_PN (none) -> 13-AC0603KRX7R6BB225CT-ND; MPN (none) -> AC0603KRX7R6BB225; Manufacturer (none) -> Yageo; Mouser_PN (none) -> 603-C0603KRX7R6BB225; Notes (none) -> Murata and TDK make no 10 V 2.2 uF X7R automotive part in 0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; Package 0603 -> (none); Placeholder PLACEHOLDER: awaiting DropOut_Resistor/DropOut_Capacitor pa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 -> (none); Temperature_Grade (none) -> AEC-Q200, -55 to +125 °C; Tolerance 10% -> ±10%
- C: footprint (none) -> DropOut_Capacitor_SMD:C_1210_3225Metric; symbol Device:C -> DropOut_Capacitor:GCM32ER71A226KE12L; Case (none) -> 1210; DigiKey_PN (none) -> 490-4797-1-ND; MPN (none) -> GCM32ER71A226KE12L; Manufacturer (none) -> Murata; Mouser_PN (none) -> 81-GCM32ER71A226KE2L; Package 1210 -> (none); Placeholder PLACEHOLDER: awaiting DropOut_Resistor/DropOut_Capacitor pa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 -> (none); Temperature_Grade (none) -> AEC-Q200, -55 to +125 °C; Tolerance 10% -> ±10%
- C: footprint (none) -> DropOut_Capacitor_SMD:C_0402_1005Metric; symbol Device:C -> DropOut_Capacitor:GCM155R71C104KA55D; Case (none) -> 0402; DigiKey_PN (none) -> 490-4759-1-ND; MPN (none) -> GCM155R71C104KA55D; Manufacturer (none) -> Murata; Mouser_PN (none) -> 81-GCM155R71C104KA5D; Package 0402 -> (none); Placeholder PLACEHOLDER: awaiting DropOut_Resistor/DropOut_Capacitor pa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 -> (none); Temperature_Grade (none) -> AEC-Q200, -55 to +125 °C; Tolerance 10% -> ±10%
- C: footprint (none) -> DropOut_Capacitor_SMD:C_0603_1608Metric; symbol Device:C -> DropOut_Capacitor:GCJ188R72A104KA01D; Case (none) -> 0603; DigiKey_PN (none) -> 490-13420-1-ND; MPN (none) -> GCJ188R72A104KA01D; Manufacturer (none) -> Murata; Mouser_PN (none) -> 81-GCJ188R72A104KA1D; Notes (none) -> Murata makes no 100 V 100 nF X7R GCM in 0603; GCJ is Murata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; Package 0603 -> (none); Placeholder PLACEHOLDER: awaiting DropOut_Resistor/DropOut_Capacitor pa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 -> (none); Temperature_Grade (none) -> AEC-Q200, -55 to +125 °C; Tolerance 10% -> ±10%
- C: footprint (none) -> DropOut_Capacitor_SMD:C_1206_3216Metric; symbol Device:C -> DropOut_Capacitor:CGA5L2X7R2A105K160AA; Case (none) -> 1206; DigiKey_PN (none) -> 445-5845-1-ND; MPN (none) -> CGA5L2X7R2A105K160AA; Manufacturer (none) -> TDK; Mouser_PN (none) -> 810-CGA5L2X7R2A105K; Package 1206 -> (none); Placeholder PLACEHOLDER: awaiting DropOut_Resistor/DropOut_Capacitor pa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 -> (none); Temperature_Grade (none) -> AEC-Q200, -55 to +125 °C; Tolerance 10% -> ±10%
- C: footprint (none) -> DropOut_Capacitor_SMD:C_0603_1608Metric; symbol Device:C -> DropOut_Capacitor:GCM188R71C105KA64D; Case (none) -> 0603; DigiKey_PN (none) -> 490-5241-1-ND; MPN (none) -> GCM188R71C105KA64D; Manufacturer (none) -> Murata; Mouser_PN (none) -> 81-GCM188R71C105K64D; Notes (none) -> No AEC-Q200 part exists in the drawn 0402 package (DigiKey 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; Package 0402 -> (none); Placeholder PLACEHOLDER: awaiting DropOut_Resistor/DropOut_Capacitor pa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 -> (none); Temperature_Grade (none) -> AEC-Q200, -55 to +125 °C; Tolerance 10% -> ±10%
- R: footprint (none) -> DropOut_Resistor_SMD:R_0402_1005Metric; symbol Device:R -> DropOut_Resistor:AC0402FR-07100KL; Case (none) -> 0402; DigiKey_PN (none) -> YAG3434CT-ND; MPN (none) -> AC0402FR-07100KL; Manufacturer (none) -> Yageo; Mouser_PN (none) -> 603-AC0402FR-07100KL; Package 0402 -> (none); Placeholder PLACEHOLDER: awaiting DropOut_Resistor/DropOut_Capacitor pa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 -> (none); Power (none) -> 1/16W; Temperature_Grade (none) -> AEC-Q200, -55 to +155 °C; Tolerance 1% -> ±1%; Voltage (none) -> 50V
- R: footprint (none) -> DropOut_Resistor_SMD:R_0603_1608Metric; symbol Device:R -> DropOut_Resistor:CRCW06030000Z0EAHP; Case (none) -> 0603; Current 2A -> (none); DigiKey_PN (none) -> 541-0.0SBCT-ND; MPN (none) -> CRCW06030000Z0EAHP; Manufacturer (none) -> Vishay; Mouser_PN (none) -> 71-CRCW06030000Z0EAH; Package 0603 -> (none); Placeholder PLACEHOLDER: awaiting DropOut_Resistor/DropOut_Capacitor pa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 -> (none); Temperature_Grade (none) -> AEC-Q200, -55 to +155 °C; Tolerance 5% -> (none)
- R: footprint (none) -> DropOut_Resistor_SMD:R_0402_1005Metric; symbol Device:R -> DropOut_Resistor:AC0402FR-0728KL; Case (none) -> 0402; DigiKey_PN (none) -> 13-AC0402FR-0728KLCT-ND; MPN (none) -> AC0402FR-0728KL; Manufacturer (none) -> Yageo; Mouser_PN (none) -> 603-AC0402FR-0728KL; Package 0402 -> (none); Placeholder PLACEHOLDER: awaiting DropOut_Resistor/DropOut_Capacitor pa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 -> (none); Power (none) -> 1/16W; Temperature_Grade (none) -> AEC-Q200, -55 to +155 °C; Tolerance 1% -> ±1%; Voltage (none) -> 50V
- R: footprint (none) -> DropOut_Resistor_SMD:R_0402_1005Metric; symbol Device:R -> DropOut_Resistor:AC0402FR-0714KL; Case (none) -> 0402; DigiKey_PN (none) -> 13-AC0402FR-0714KLCT-ND; MPN (none) -> AC0402FR-0714KL; Manufacturer (none) -> Yageo; Mouser_PN (none) -> 603-AC0402FR-0714KL; Package 0402 -> (none); Placeholder PLACEHOLDER: awaiting DropOut_Resistor/DropOut_Capacitor pa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 -> (none); Power (none) -> 1/16W; Temperature_Grade (none) -> AEC-Q200, -55 to +155 °C; Tolerance 1% -> ±1%; Voltage (none) -> 50V
- R: footprint (none) -> DropOut_Resistor_SMD:R_0402_1005Metric; symbol Device:R -> DropOut_Resistor:AC0402JR-074K7L; Case (none) -> 0402; DigiKey_PN (none) -> 311-4.7KLBCT-ND; MPN (none) -> AC0402JR-074K7L; Manufacturer (none) -> Yageo; Mouser_PN (none) -> 603-AC0402JR-074K7L; Package 0402 -> (none); Placeholder PLACEHOLDER: awaiting DropOut_Resistor/DropOut_Capacitor pa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 -> (none); Power (none) -> 1/16W; Temperature_Grade (none) -> AEC-Q200, -55 to +155 °C; Tolerance 5% -> ±5%; Voltage (none) -> 50V
- R: footprint (none) -> DropOut_Resistor_SMD:R_0402_1005Metric; symbol Device:R -> DropOut_Resistor:AC0402JR-070RL; Case (none) -> 0402; DigiKey_PN (none) -> 311-0.0LBCT-ND; MPN (none) -> AC0402JR-070RL; Manufacturer (none) -> Yageo; Mouser_PN (none) -> 603-AC0402JR-070RL; Package 0402 -> (none); Placeholder PLACEHOLDER: awaiting DropOut_Resistor/DropOut_Capacitor pa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 -> (none); Temperature_Grade (none) -> AEC-Q200, -55 to +155 °C; Tolerance 5% -> (none)
- TP: value TP_VDDAU_AON -> TestPoint_Pad_D1.0mm; footprint (none) -> DropOut_TestPoint:TestPoint_Pad_D1.0mm; symbol Connector:TestPoint -> DropOut_Connector:TestPoint_Pad_D1.0mm; DigiKey_PN (none) -> -; MPN (none) -> TestPoint_Pad_D1.0mm; Manufacturer (none) -> DropOut; Mouser_PN (none) -> -; Notes (none) -> PCB copper only; nothing to order. Excluded from BOM and po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; Placeholder PLACEHOLDER: awaiting DropOut test-point part (library brie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 -> (none); Type 1mm pad -> (none)
- TP: value TP_1V5_CORE -> TestPoint_Pad_D1.0mm; footprint (none) -> DropOut_TestPoint:TestPoint_Pad_D1.0mm; symbol Connector:TestPoint -> DropOut_Connector:TestPoint_Pad_D1.0mm; DigiKey_PN (none) -> -; MPN (none) -> TestPoint_Pad_D1.0mm; Manufacturer (none) -> DropOut; Mouser_PN (none) -> -; Notes (none) -> PCB copper only; nothing to order. Excluded from BOM and po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; Placeholder PLACEHOLDER: awaiting DropOut test-point part (library brie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 -> (none); Type 1mm pad -> (none)
- TP: value TP_3V3_MAIN -> TestPoint_Pad_D1.0mm; footprint (none) -> DropOut_TestPoint:TestPoint_Pad_D1.0mm; symbol Connector:TestPoint -> DropOut_Connector:TestPoint_Pad_D1.0mm; DigiKey_PN (none) -> -; MPN (none) -> TestPoint_Pad_D1.0mm; Manufacturer (none) -> DropOut; Mouser_PN (none) -> -; Notes (none) -> PCB copper only; nothing to order. Excluded from BOM and po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; Placeholder PLACEHOLDER: awaiting DropOut test-point part (library brie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 -> (none); Type 1mm pad -> (none)
- TP: value TP_INH -> TestPoint_Pad_D1.0mm; footprint (none) -> DropOut_TestPoint:TestPoint_Pad_D1.0mm; symbol Connector:TestPoint -> DropOut_Connector:TestPoint_Pad_D1.0mm; DigiKey_PN (none) -> -; MPN (none) -> TestPoint_Pad_D1.0mm; Manufacturer (none) -> DropOut; Mouser_PN (none) -> -; Notes (none) -> PCB copper only; nothing to order. Excluded from BOM and po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; Placeholder PLACEHOLDER: awaiting DropOut test-point part (library brie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 -> (none); Type 1mm pad -> (none)
- TP: value TP_GND -> S1751-46R; footprint (none) -> DropOut_TestPoint:TestPoint_Harwin_S1751; symbol Connector:TestPoint -> DropOut_Connector:S1751-46R; DigiKey_PN (none) -> 952-1478-1-ND; MPN (none) -> S1751-46R; Manufacturer (none) -> Harwin; Mouser_PN (none) -> 855-S1751-46R; Notes (none) -> Ground test point (probe loop) for a scope ground spring or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; Placeholder PLACEHOLDER: awaiting DropOut test-point part (library brie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 -> (none); Temperature_Grade (none) -> -55 to +125 °C; Type probe loop -> (none)
- TP: value TP_1V5_EN -> TestPoint_Pad_D1.0mm; footprint (none) -> DropOut_TestPoint:TestPoint_Pad_D1.0mm; symbol Connector:TestPoint -> DropOut_Connector:TestPoint_Pad_D1.0mm; DigiKey_PN (none) -> -; MPN (none) -> TestPoint_Pad_D1.0mm; Manufacturer (none) -> DropOut; Mouser_PN (none) -> -; Notes (none) -> PCB copper only; nothing to order. Excluded from BOM and po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; Placeholder PLACEHOLDER: awaiting DropOut test-point part (library brie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 -> (none); Type 1mm pad -> (none)
- TP: value TP_VBAT_FILT -> TestPoint_Pad_D1.0mm; footprint (none) -> DropOut_TestPoint:TestPoint_Pad_D1.0mm; symbol Connector:TestPoint -> DropOut_Connector:TestPoint_Pad_D1.0mm; DigiKey_PN (none) -> -; MPN (none) -> TestPoint_Pad_D1.0mm; Manufacturer (none) -> DropOut; Mouser_PN (none) -> -; Notes (none) -> PCB copper only; nothing to order. Excluded from BOM and po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; Placeholder PLACEHOLDER: awaiting DropOut test-point part (library brie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 -> (none); Type 1mm pad -> (none)
- TP: value TP_RESET_L -> TestPoint_Pad_D1.0mm; footprint (none) -> DropOut_TestPoint:TestPoint_Pad_D1.0mm; symbol Connector:TestPoint -> DropOut_Connector:TestPoint_Pad_D1.0mm; DigiKey_PN (none) -> -; MPN (none) -> TestPoint_Pad_D1.0mm; Manufacturer (none) -> DropOut; Mouser_PN (none) -> -; Notes (none) -> PCB copper only; nothing to order. Excluded from BOM and po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; Placeholder PLACEHOLDER: awaiting DropOut test-point part (library brie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 -> (none); Type 1mm pad -> (none)
