File: sheets/mcu-nvm.kicad_sch (KiCad schematic)
At the start: 0 parts

Commit message: Schematic capture: MCU and NVM (p4), connectors (p9); ERC clean
Page 4: S32K344 in eight boxed units. The supply unit has decoupling per
NXP HDG Rev E2 Table 2; each port unit shows its pin plan and firmware
notes (D-14 as adopted). Pins were checked against NXP's IOMUX table:
EMAC RMII per NXP's TJA1100 use case, LPSPI4 switch chain, LPSPI2 log
flash, LPI2C0 telemetry, ADC1/ADC2 inputs, EIRQ fault lines, SWD and an
LPUART0 debug port. Also the IS25LP032D flash, the Cortex 10-pin header
and the I2C pull-ups.

Page 9: placeholder battery, return, T1S and MX150 output connectors
(all TBD selections), mirrored with pin 1 at the top (D-43), and the
PWR_FLAGs for nets entering the board.

ERC: 0 violations. 17 items are excluded in node60.kicad_pro, each with
its reason (D-52): parallel output pins typed power output in the
library (to be retyped there), and two LAN8670 pins tied to VSS per the
datasheet.

Co-Authored-By: Claude Opus 5.5 <noreply@anthropic.com>
Parts:
- added C (x18): 100nF, symbol Device:C
- added C: 4.7uF, symbol Device:C
- added C: 1uF, symbol Device:C
- added C: 2.2uF, symbol Device:C
- added C: 10uF, symbol Device:C
- added C: 220nF, symbol Device:C
- added J: FTSH-105-01-L-DV-K, DropOut_Connector_Samtec:Samtec_FTSH-105-01-x-DV_2x05_P1.27mm_Vertical_SMD, symbol DropOut_Connector:FTSH-105-01-L-DV-K
- added R (x2): 2.2k, symbol Device:R
- added R (x5): 10k, symbol Device:R
- added TP: TP_SPI4_SWITCH_MISO, symbol Connector:TestPoint
- added TP: TP_GND, symbol Connector:TestPoint
- added TP: TP_1V1_MCU_V11, symbol Connector:TestPoint
- added TP: TP_SPI2_FLASH_CS_L, symbol Connector:TestPoint
- added TP: TP_I2C0_TELEMETRY_SDA, symbol Connector:TestPoint
- added TP: TP_I2C0_TELEMETRY_SCL, symbol Connector:TestPoint
- added TP: TP_SPI4_SWITCH_CS_L, symbol Connector:TestPoint
- added TP: TP_SPI4_SWITCH_MOSI, symbol Connector:TestPoint
- added TP: TP_UART0_DEBUG_TX, symbol Connector:TestPoint
- added TP: TP_SPI2_FLASH_SCK, symbol Connector:TestPoint
- added TP: TP_UART0_DEBUG_RX, symbol Connector:TestPoint
- added TP: TP_SPI4_SWITCH_SCK, symbol Connector:TestPoint
- added U: S32K344EHT1MMMST, DropOut_Package_BGA:NXP_LFBGA-257_14x14mm_Layout17x17_P0.8mm, symbol DropOut_MCU_NXP:S32K344EHT1MMMST
Connections:
- new net 1V1_MCU_V11: C.1, C.1, C.1, C.1, C.1, TP.1, U.H9 (V11), U.J10 (V11), U.J8 (V11), U.K9 (V11)
- new net 1V5_CORE: C.1, C.1, C.1, C.1, C.1, U.H10 (V15), U.H8 (V15), U.K10 (V15), U.K8 (V15)
- new net 2V5_MCU_V25: C.1, U.J7 (V25)
- new net 3V3_MAIN: C.1, C.1, C.1, C.1, C.1, C.1, C.1, C.1, C.1, C.1, C.1, C.1, J.1 (Pin_1), R.1, R.1, R.1, R.1, R.1, R.1, U.8 (VCC), U.D14 (VDD_HV_A), U.G10 (VDD_HV_A), U.H6 (VREFH), U.H7 (VDD_HV_A), U.K11 (VDD_HV_A), U.L8 (VDD_HV_A), U.N4 (VDD_HV_B), U.R10 (VDD_HV_B), U.R7 (VDD_HV_B)
- new net BATT_MON: U.B1 (PTA18)
- new net FLASH_HOLD_L: R.2, U.7 (~{HOLD}/~{RESET}/IO3)
- new net FLASH_WP_L: R.2, U.3 (~{WP}/IO2)
- new net GND: C.2, C.2, C.2, C.2, C.2, C.2, C.2, C.2, C.2, C.2, C.2, C.2, C.2, C.2, C.2, C.2, C.2, C.2, C.2, C.2, C.2, C.2, C.2, J.3 (Pin_3), J.5 (Pin_5), J.9 (Pin_9), R.2, TP.1, U.4 (GND), U.B16 (VSS), U.B2 (VSS), U.D4 (VSS), U.D9 (VSS), U.G11 (VSS), U.G7 (VSS), U.J1 (VSS), U.J14 (VSS), U.J4 (VSS), U.J6 (VREFL), U.J9 (VSS), U.L11 (VSS), U.L7 (VSS), U.P14 (VSS), U.P4 (VSS), U.T10 (VSS), U.T16 (VSS), U.T2 (VSS), U.T7 (VSS)
- new net I2C0_TELEMETRY_SCL: R.2, TP.1, U.M4 (PTD14)
- new net I2C0_TELEMETRY_SDA: R.2, TP.1, U.P5 (PTD13)
- new net LM_FLT_L: U.B11 (PTE6)
- new net MDIO0_T1S_MDC: U.N3 (PTD17)
- new net MDIO0_T1S_MDIO: U.P2 (PTD16)
- new net NTC_RSENSE: U.C1 (PTA19)
- new net NTC_SW1: U.E4 (PTA20)
- new net NTC_SW2: U.F9 (PTE21)
- new net NTC_SW3: U.B9 (PTE22)
- new net RESET_L: J.10 (Pin_10), U.A3 (PTA5/~{RESET})
- new net RMII0_T1S_CRS_DV: U.R6 (PTC17)
- new net RMII0_T1S_REF_CLK: U.U6 (PTD11)
- new net RMII0_T1S_RXD0: U.T8 (PTC1)
- new net RMII0_T1S_RXD1: U.U7 (PTC0)
- new net RMII0_T1S_RX_ER: U.P6 (PTC16)
- new net RMII0_T1S_TXD0: U.U4 (PTD7)
- new net RMII0_T1S_TXD1: U.T4 (PTC2)
- new net RMII0_T1S_TX_EN: U.R5 (PTD12)
- new net SPI2_FLASH_CS_L: R.2, TP.1, U.1 (~{CE}), U.E1 (PTE11)
- new net SPI2_FLASH_MISO: U.2 (SO/IO1), U.C2 (PTE16)
- new net SPI2_FLASH_MOSI: U.5 (SI/IO0), U.C6 (PTF2)
- new net SPI2_FLASH_SCK: TP.1, U.6 (SCK), U.D2 (PTE15)
- new net SPI4_SWITCH_CS_L: TP.1, U.A14 (PTB8)
- new net SPI4_SWITCH_MISO: TP.1, U.C17 (PTB11)
- new net SPI4_SWITCH_MOSI: TP.1, U.C15 (PTB9)
- new net SPI4_SWITCH_SCK: TP.1, U.D15 (PTB10)
- new net SW1_FLT_L: U.B5 (PTE0)
- new net SW1_SNS: U.A7 (PTA12/CLKOUT_STANDBY)
- new net SW2_FLT_L: U.A5 (PTE1)
- new net SW2_SNS: U.A9 (PTA13)
- new net SW3_FLT_L: U.B10 (PTE2)
- new net SW3_SNS: U.A10 (PTA14)
- new net SWD_CLK: J.4 (Pin_4), R.1, U.F7 (PTC4/JTAG_TCK/SWD_CLK)
- new net SWD_DIO: J.2 (Pin_2), R.2, U.F6 (PTA4/JTAG_TMS/SWD_DIO)
- new net SWD_SWO: J.6 (Pin_6), U.G8 (PTA10/JTAG_TDO/TRACEnoETM_SWO)
- new net T1S_IRQ_L: U.B3 (PTA9)
- new net TMP175_ALERT_L: U.A11 (PTA15)
- new net UART0_DEBUG_RX: TP.1, U.D17 (PTA2)
- new net UART0_DEBUG_TX: TP.1, U.E16 (PTA3)
- no-connect marks 0 -> 182
Other:
- note added: "ADC: SW1..3_SNS on ADC1_P0/P1/P4; BATT_MON ADC2_P0; NTC_RSENSE ADC2_P1; NTC_SW1 ADC2_P2. EIRQ17 = PHY IRQ (falling edge), EIRQ23 = TMP175 ALERT. PTA5 stays RESET_B (default function)."
- note added: "All PTG pins unused: no-connect."
- note added: "DESIGN NOTES (S32K3xx data sheet; S32K3 Hardware Design Guidelines Rev E2; Node60 compute page) RELEASE-BLOCKING (GATE-MCU-01): ball map from the library symbol (NXP IOMUX attachment, Nov 2025). Check every ball and ALT setting here against the S32K344EHT1MMMST package before layout. The pin table above each unit is the plan. Supplies: VDD_HV_A = VDD_HV_B = VREFH = 3V3_MAIN, V15 = 1V5_CORE (U303)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"
- note added: "Diagnostic log flash, LPSPI2 (U402, DEC-011)"
- note added: "EXTAL/XTAL: no crystal in Rev A (FIRC clocks the core; RMII uses the 50 MHz oscillator). VREFL ties to VSS. V11 and V25 are internal regulator outputs: decoupling only, no loads."
- note added: "Fault lines are open drain with pull-ups at the source; EIRQ on falling edge. NTC_SW2/3 on ADC2_P3/P4."
- note added: "I2C0 telemetry pull-ups (bus: U202, U203)"
- note added: "LPSPI4 master, mode per TPS2HCS08 datasheet, 3 x 24-bit frames per CS with CRC. PCS0 must idle high from reset: switches keep all channels off until configured."
- note added: "PTA (U401B): ADC1 output-current SNS, ADC2 temperatures and BATT_MON, SWD, RESET_B, LPUART0 debug, EIRQ"
- note added: "PTB (U401C): LPSPI4: TPS2HCS08 daisy chain"
- note added: "PTC (U401D): EMAC RMII receive, TXD1, SWD clock"
- note added: "PTD (U401E): EMAC RMII transmit, MDIO, LPI2C0 telemetry"
- note added: "PTE (U401F): Fault inputs (EIRQ), LPSPI2 flash, ADC2 temperatures"
- note added: "PTF (U401G): LPSPI2 flash MOSI"
- note added: "PTG (U401H): Unused"
- note added: "RMII REF_CLK enters on EMAC TX_CLK (RM: 'EMAC transmitter clock / RMII clock'). LPI2C0 standard/fast mode: INA228 0x40, TMP175 0x48."
- note added: "RMII pins follow NXP's TJA1100 RMII use case (IOMUX 'Ethernet use cases' sheet)."
- note added: "S32K344 supplies and decoupling (U401A), NXP HDG Rev E2 Table 2"
- note added: "SWD debug header, 2x5 1.27 mm Cortex (J401) and LPUART0 test pads"
- note added: "Test points"
- note added: "Unused pins: no-connect (default GPIO input, disabled)."
- note added: "V15 (1.5 V core supply from U303)"
- note added: "VDD_HV_A x5, VDD_HV_B x3, VREFH: 100nF per ball, 1uF at VREFH, 10uF bulk (one bulk: HV_A and HV_B share 3V3_MAIN)"
- title: Node60 -> Node60 · C · MCU and NVM (p4)

Commit message: Swap placeholders for merged DropOut library parts
Library bumped to ce98ecf (PRs #15, #16, #18, #19, #20, #21 merged).
Now real parts: IAUTN08S5N012LATMA1 (Q201-Q204, dual gate: G_ON and
G_LIN both driven), CSS2725FTL250 (R201, 2-terminal: sense nets are
VBAT_D / VBAT_Q2D with Kelvin taps from the pads in layout),
TPS7B8133QWDRVRQ1 (U301, COUT 2.2uF per its 1-200 uF requirement),
NCU18XH103F6SRB (RT201, RT601-801), Wurth 74438356022HT / 74438356010HT
buck inductors and Harwin S1751-46R GND loops (user's picks 2026-10-23),
1 mm pad test points and DT13-2P output headers. The library pin-type
fixes cut the ERC exclusions from 17 to 2. parts.yaml records the
library symbols; the library tables list the new libraries.

Co-Authored-By: Claude Opus 5.5 <noreply@anthropic.com>
Parts:
- TP: Placeholder PLACEHOLDER: test point part pending (library brief 03) -> PLACEHOLDER: awaiting DropOut test-point part (library brie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
Changed lines of the file:
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@@
 			)
 		)
-		(property "Placeholder" "PLACEHOLDER: test point part pending (library brief 03)"
+		(property "Manufacturer" ""
+			(at 170.18 355.6 0)
+			(effects
+				(font
+					(size 1.27 1.27)
+				)
+				(hide yes)
+			)
+		)
+		(property "DigiKey_PN" ""
+			(at 170.18 355.6 0)
+			(effects
+				(font
+					(size 1.27 1.27)
+				)
+				(hide yes)
+			)
+		)
+		(property "Mouser_PN" ""
+			(at 170.18 355.6 0)
+			(effects
+				(font
+					(size 1.27 1.27)
+				)
+				(hide yes)
+			)
+		)
+		(property "Placeholder" "PLACEHOLDER: awaiting DropOut test-point part (library brief 03-connectors-testpoints)"
 			(at 170.18 355.6 0)
 			(effects
@@
 			)
 		)
-		(property "Placeholder" "PLACEHOLDER: test point part pending (library brief 03)"
+		(property "Manufacturer" ""
 			(at 193.04 355.6 0)
 			(effects
+				(font
+					(size 1.27 1.27)
+				)
+				(hide yes)
+			)
+		)
+		(property "DigiKey_PN" ""
+			(at 193.04 355.6 0)
+			(effects
+				(font
+					(size 1.27 1.27)
+				)
+				(hide yes)
+			)
+		)
+		(property "Mouser_PN" ""
+			(at 193.04 355.6 0)
+			(effects
+				(font
+					(size 1.27 1.27)
+				)
+				(hide yes)
+			)
+		)
+		(property "Placeholder" "PLACEHOLDER: awaiting DropOut test-point part (library brief 03-connectors-testpoints)"
+			(at 193.04 355.6 0)
+			(effects

Commit message: Swap all resistors, capacitors and test points for DropOut parts
Library bumped to 752b63c (PR #22: 83 AEC-Q200 chip resistors and MLCCs,
PR #24: passive symbol layout). Each passive is now a real part, chosen
by rule: exact value and dielectric, tolerance and voltage at least as
good, the drawn package else the next larger, then manufacturer order;
the other built sources stay in the library as alternates.

Where the library has no part in the drawn package: 10nF C0G, 4.7nF C0G,
1uF 16V and 470nF 16V 0402 -> 0603; 68nF C0G, 100nF C0G and 10uF 16V
0805 -> 1206; 32k 1% -> 0.1% (TNPW060332K0BEEA); CCAP 1uF 50V (not built)
-> 1uF 100V 1206. 0R debug links on regulator outputs use the 5 A
CRCW06030000Z0EAHP jumper.

Also fixes test points: f9af1d2 described them as swapped, but they were
still stock symbols. They are now TestPoint_Pad_D1.0mm (signals) and
Harwin S1751-46R (GND loops).

Only placeholders left: L201 / C208 (EMI filter, TBD) and J901-J903.

Co-Authored-By: Claude Opus 5.5 <noreply@anthropic.com>
Parts:
- C: footprint (none) -> DropOut_Capacitor_SMD:C_0402_1005Metric; symbol Device:C -> DropOut_Capacitor:GCM155R71C104KA55D; Case (none) -> 0402; DigiKey_PN (none) -> 490-4759-1-ND; MPN (none) -> GCM155R71C104KA55D; Manufacturer (none) -> Murata; Mouser_PN (none) -> 81-GCM155R71C104KA5D; Package 0402 -> (none); Placeholder PLACEHOLDER: awaiting DropOut_Resistor/DropOut_Capacitor pa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 -> (none); Temperature_Grade (none) -> AEC-Q200, -55 to +125 °C; Tolerance 10% -> ±10%
- C: footprint (none) -> DropOut_Capacitor_SMD:C_0805_2012Metric; symbol Device:C -> DropOut_Capacitor:GCM21BR71C475KA73L; Case (none) -> 0805; DigiKey_PN (none) -> 490-5332-1-ND; MPN (none) -> GCM21BR71C475KA73L; Manufacturer (none) -> Murata; Mouser_PN (none) -> 81-GCM21BR71C475KA3L; Notes (none) -> Murata's lowest rating for this value in GCM21B X7R is 16 V.; Package 0805 -> (none); Placeholder PLACEHOLDER: awaiting DropOut_Resistor/DropOut_Capacitor pa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 -> (none); Temperature_Grade (none) -> AEC-Q200, -55 to +125 °C; Tolerance 10% -> ±10%; Voltage 10V -> 16V
- C: footprint (none) -> DropOut_Capacitor_SMD:C_0603_1608Metric; symbol Device:C -> DropOut_Capacitor:GCM188R71C105KA64D; Case (none) -> 0603; DigiKey_PN (none) -> 490-5241-1-ND; MPN (none) -> GCM188R71C105KA64D; Manufacturer (none) -> Murata; Mouser_PN (none) -> 81-GCM188R71C105K64D; Notes (none) -> No AEC-Q200 part exists in the drawn 0402 package (DigiKey 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; Package 0402 -> (none); Placeholder PLACEHOLDER: awaiting DropOut_Resistor/DropOut_Capacitor pa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 -> (none); Temperature_Grade (none) -> AEC-Q200, -55 to +125 °C; Tolerance 10% -> ±10%
- C: footprint (none) -> DropOut_Capacitor_SMD:C_0603_1608Metric; symbol Device:C -> DropOut_Capacitor:AC0603KRX7R6BB225; Case (none) -> 0603; DigiKey_PN (none) -> 13-AC0603KRX7R6BB225CT-ND; MPN (none) -> AC0603KRX7R6BB225; Manufacturer (none) -> Yageo; Mouser_PN (none) -> 603-C0603KRX7R6BB225; Notes (none) -> Murata and TDK make no 10 V 2.2 uF X7R automotive part in 0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; Package 0603 -> (none); Placeholder PLACEHOLDER: awaiting DropOut_Resistor/DropOut_Capacitor pa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 -> (none); Temperature_Grade (none) -> AEC-Q200, -55 to +125 °C; Tolerance 10% -> ±10%
- C: footprint (none) -> DropOut_Capacitor_SMD:C_1206_3216Metric; symbol Device:C -> DropOut_Capacitor:GCM31CR71C106KA64L; Case (none) -> 1206; DigiKey_PN (none) -> 490-4793-1-ND; MPN (none) -> GCM31CR71C106KA64L; Manufacturer (none) -> Murata; Mouser_PN (none) -> 81-GCM31CR71C106KA4L; Notes (none) -> No AEC-Q200 10 uF 16 V X7R part exists in the drawn 0805 pa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; Package 0805 -> (none); Placeholder PLACEHOLDER: awaiting DropOut_Resistor/DropOut_Capacitor pa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 -> (none); Temperature_Grade (none) -> AEC-Q200, -55 to +125 °C; Tolerance 10% -> ±10%
- C: footprint (none) -> DropOut_Capacitor_SMD:C_0402_1005Metric; symbol Device:C -> DropOut_Capacitor:GCM155R71C224KE02D; Case (none) -> 0402; DigiKey_PN (none) -> 490-10671-1-ND; MPN (none) -> GCM155R71C224KE02D; Manufacturer (none) -> Murata; Mouser_PN (none) -> 81-GCM155R71C224KE2D; Package 0402 -> (none); Placeholder PLACEHOLDER: awaiting DropOut_Resistor/DropOut_Capacitor pa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 -> (none); Temperature_Grade (none) -> AEC-Q200, -55 to +125 °C; Tolerance 10% -> ±10%
- R: footprint (none) -> DropOut_Resistor_SMD:R_0402_1005Metric; symbol Device:R -> DropOut_Resistor:AC0402JR-072K2L; Case (none) -> 0402; DigiKey_PN (none) -> YAG3536CT-ND; MPN (none) -> AC0402JR-072K2L; Manufacturer (none) -> Yageo; Mouser_PN (none) -> 603-AC0402JR-072K2L; Package 0402 -> (none); Placeholder PLACEHOLDER: awaiting DropOut_Resistor/DropOut_Capacitor pa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 -> (none); Power (none) -> 1/16W; Temperature_Grade (none) -> AEC-Q200, -55 to +155 °C; Tolerance 5% -> ±5%; Voltage (none) -> 50V
- R: footprint (none) -> DropOut_Resistor_SMD:R_0402_1005Metric; symbol Device:R -> DropOut_Resistor:AC0402JR-0710KL; Case (none) -> 0402; DigiKey_PN (none) -> YAG3517CT-ND; MPN (none) -> AC0402JR-0710KL; Manufacturer (none) -> Yageo; Mouser_PN (none) -> 603-AC0402JR-0710KL; Package 0402 -> (none); Placeholder PLACEHOLDER: awaiting DropOut_Resistor/DropOut_Capacitor pa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 -> (none); Power (none) -> 1/16W; Temperature_Grade (none) -> AEC-Q200, -55 to +155 °C; Tolerance 5% -> ±5%; Voltage (none) -> 50V
- TP: value TP_SPI4_SWITCH_MISO -> TestPoint_Pad_D1.0mm; footprint (none) -> DropOut_TestPoint:TestPoint_Pad_D1.0mm; symbol Connector:TestPoint -> DropOut_Connector:TestPoint_Pad_D1.0mm; DigiKey_PN (none) -> -; MPN (none) -> TestPoint_Pad_D1.0mm; Manufacturer (none) -> DropOut; Mouser_PN (none) -> -; Notes (none) -> PCB copper only; nothing to order. Excluded from BOM and po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; Placeholder PLACEHOLDER: awaiting DropOut test-point part (library brie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 -> (none); Type 1mm pad -> (none)
- TP: value TP_GND -> S1751-46R; footprint (none) -> DropOut_TestPoint:TestPoint_Harwin_S1751; symbol Connector:TestPoint -> DropOut_Connector:S1751-46R; DigiKey_PN (none) -> 952-1478-1-ND; MPN (none) -> S1751-46R; Manufacturer (none) -> Harwin; Mouser_PN (none) -> 855-S1751-46R; Notes (none) -> Ground test point (probe loop) for a scope ground spring or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; Placeholder PLACEHOLDER: awaiting DropOut test-point part (library brie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 -> (none); Temperature_Grade (none) -> -55 to +125 °C; Type probe loop -> (none)
- TP: value TP_1V1_MCU_V11 -> TestPoint_Pad_D1.0mm; footprint (none) -> DropOut_TestPoint:TestPoint_Pad_D1.0mm; symbol Connector:TestPoint -> DropOut_Connector:TestPoint_Pad_D1.0mm; DigiKey_PN (none) -> -; MPN (none) -> TestPoint_Pad_D1.0mm; Manufacturer (none) -> DropOut; Mouser_PN (none) -> -; Notes (none) -> PCB copper only; nothing to order. Excluded from BOM and po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; Placeholder PLACEHOLDER: awaiting DropOut test-point part (library brie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 -> (none); Type 1mm pad -> (none)
- TP: value TP_SPI2_FLASH_CS_L -> TestPoint_Pad_D1.0mm; footprint (none) -> DropOut_TestPoint:TestPoint_Pad_D1.0mm; symbol Connector:TestPoint -> DropOut_Connector:TestPoint_Pad_D1.0mm; DigiKey_PN (none) -> -; MPN (none) -> TestPoint_Pad_D1.0mm; Manufacturer (none) -> DropOut; Mouser_PN (none) -> -; Notes (none) -> PCB copper only; nothing to order. Excluded from BOM and po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; Placeholder PLACEHOLDER: awaiting DropOut test-point part (library brie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 -> (none); Type 1mm pad -> (none)
- TP: value TP_I2C0_TELEMETRY_SDA -> TestPoint_Pad_D1.0mm; footprint (none) -> DropOut_TestPoint:TestPoint_Pad_D1.0mm; symbol Connector:TestPoint -> DropOut_Connector:TestPoint_Pad_D1.0mm; DigiKey_PN (none) -> -; MPN (none) -> TestPoint_Pad_D1.0mm; Manufacturer (none) -> DropOut; Mouser_PN (none) -> -; Notes (none) -> PCB copper only; nothing to order. Excluded from BOM and po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; Placeholder PLACEHOLDER: awaiting DropOut test-point part (library brie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 -> (none); Type 1mm pad -> (none)
- TP: value TP_I2C0_TELEMETRY_SCL -> TestPoint_Pad_D1.0mm; footprint (none) -> DropOut_TestPoint:TestPoint_Pad_D1.0mm; symbol Connector:TestPoint -> DropOut_Connector:TestPoint_Pad_D1.0mm; DigiKey_PN (none) -> -; MPN (none) -> TestPoint_Pad_D1.0mm; Manufacturer (none) -> DropOut; Mouser_PN (none) -> -; Notes (none) -> PCB copper only; nothing to order. Excluded from BOM and po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; Placeholder PLACEHOLDER: awaiting DropOut test-point part (library brie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 -> (none); Type 1mm pad -> (none)
- TP: value TP_SPI4_SWITCH_CS_L -> TestPoint_Pad_D1.0mm; footprint (none) -> DropOut_TestPoint:TestPoint_Pad_D1.0mm; symbol Connector:TestPoint -> DropOut_Connector:TestPoint_Pad_D1.0mm; DigiKey_PN (none) -> -; MPN (none) -> TestPoint_Pad_D1.0mm; Manufacturer (none) -> DropOut; Mouser_PN (none) -> -; Notes (none) -> PCB copper only; nothing to order. Excluded from BOM and po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; Placeholder PLACEHOLDER: awaiting DropOut test-point part (library brie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 -> (none); Type 1mm pad -> (none)
- TP: value TP_SPI4_SWITCH_MOSI -> TestPoint_Pad_D1.0mm; footprint (none) -> DropOut_TestPoint:TestPoint_Pad_D1.0mm; symbol Connector:TestPoint -> DropOut_Connector:TestPoint_Pad_D1.0mm; DigiKey_PN (none) -> -; MPN (none) -> TestPoint_Pad_D1.0mm; Manufacturer (none) -> DropOut; Mouser_PN (none) -> -; Notes (none) -> PCB copper only; nothing to order. Excluded from BOM and po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; Placeholder PLACEHOLDER: awaiting DropOut test-point part (library brie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 -> (none); Type 1mm pad -> (none)
- TP: value TP_UART0_DEBUG_TX -> TestPoint_Pad_D1.0mm; footprint (none) -> DropOut_TestPoint:TestPoint_Pad_D1.0mm; symbol Connector:TestPoint -> DropOut_Connector:TestPoint_Pad_D1.0mm; DigiKey_PN (none) -> -; MPN (none) -> TestPoint_Pad_D1.0mm; Manufacturer (none) -> DropOut; Mouser_PN (none) -> -; Notes (none) -> PCB copper only; nothing to order. Excluded from BOM and po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; Placeholder PLACEHOLDER: awaiting DropOut test-point part (library brie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 -> (none); Type 1mm pad -> (none)
- TP: value TP_SPI2_FLASH_SCK -> TestPoint_Pad_D1.0mm; footprint (none) -> DropOut_TestPoint:TestPoint_Pad_D1.0mm; symbol Connector:TestPoint -> DropOut_Connector:TestPoint_Pad_D1.0mm; DigiKey_PN (none) -> -; MPN (none) -> TestPoint_Pad_D1.0mm; Manufacturer (none) -> DropOut; Mouser_PN (none) -> -; Notes (none) -> PCB copper only; nothing to order. Excluded from BOM and po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; Placeholder PLACEHOLDER: awaiting DropOut test-point part (library brie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 -> (none); Type 1mm pad -> (none)
- TP: value TP_UART0_DEBUG_RX -> TestPoint_Pad_D1.0mm; footprint (none) -> DropOut_TestPoint:TestPoint_Pad_D1.0mm; symbol Connector:TestPoint -> DropOut_Connector:TestPoint_Pad_D1.0mm; DigiKey_PN (none) -> -; MPN (none) -> TestPoint_Pad_D1.0mm; Manufacturer (none) -> DropOut; Mouser_PN (none) -> -; Notes (none) -> PCB copper only; nothing to order. Excluded from BOM and po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; Placeholder PLACEHOLDER: awaiting DropOut test-point part (library brie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 -> (none); Type 1mm pad -> (none)
- TP: value TP_SPI4_SWITCH_SCK -> TestPoint_Pad_D1.0mm; footprint (none) -> DropOut_TestPoint:TestPoint_Pad_D1.0mm; symbol Connector:TestPoint -> DropOut_Connector:TestPoint_Pad_D1.0mm; DigiKey_PN (none) -> -; MPN (none) -> TestPoint_Pad_D1.0mm; Manufacturer (none) -> DropOut; Mouser_PN (none) -> -; Notes (none) -> PCB copper only; nothing to order. Excluded from BOM and po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; Placeholder PLACEHOLDER: awaiting DropOut test-point part (library brie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 -> (none); Type 1mm pad -> (none)

Commit message: Schematic: LHI to the MCU, current notes, net-name map
- LHI on all three TPS2HCS08 is now SW_LHI from S32K344 PTE4 (the
  architecture's GPIO list), still held low by the 10k pull-downs
  through reset.
- Page 4 cites NXP HDG Rev E2 Table 33 for unused GPIO, EXTAL/XTAL and
  the RESET_B pull-up instead of an open 'confirm' note.
- Copper notes for the 10 A output paths (p6) and the 60 A path (p2,
  p9), as IPC-2221 starting estimates to confirm with IPC-2152.
- interfaces.mdx maps the architecture's signal names to the schematic
  nets (RESET_L, T1S_IRQ_L, *_FLT_L, SPI4/SPI2/I2C0 buses).

Co-Authored-By: Claude Opus 5.5 <noreply@anthropic.com>
Connections:
- net SW_LHI: now reaches U.G6 (PTE4)
- no-connect marks 182 -> 181
Other:
- note added: "Fault lines are open drain with pull-ups at the source; EIRQ on falling edge. NTC_SW2/3 on ADC2_P3/P4. SW_LHI (PTE4) output, driven low; never asserted in normal operation."
- note removed: "Fault lines are open drain with pull-ups at the source; EIRQ on falling edge. NTC_SW2/3 on ADC2_P3/P4."
Changed lines of the file:
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@@
 		)
 	)
-	(no_connect
-		(at 505.46 210.82)
+	(wire
+		(pts
+			(xy 505.46 210.82)
+			(xy 502.92 210.82)
+		)
+		(stroke
+			(width 0)
+			(type default)
+		)
+	)
+	(hierarchical_label "SW_LHI"
+		(shape output)
+		(at 502.92 210.82 180)
+		(effects
+			(font
+				(size 1.27 1.27)
+			)
+			(justify right)
+		)
 	)
 	(no_connect
@@
 		)
 	)
-	(text "Fault lines are open drain with pull-ups at the source; EIRQ on falling edge.\nNTC_SW2/3 on ADC2_P3/P4."
+	(text "Fault lines are open drain with pull-ups at the source; EIRQ on falling edge.\nNTC_SW2/3 on ADC2_P3/P4. SW_LHI (PTE4) output, driven low; never asserted in normal operation."
 		(exclude_from_sim no)
 		(at 457.2 248.92 0)
@@
 		)
 	)
-	(text "DESIGN NOTES (S32K3xx data sheet; S32K3 Hardware Design Guidelines Rev E2; Node60 compute page)\nRELEASE-BLOCKING (GATE-MCU-01): ball map from the library symbol (NXP IOMUX attachment, Nov 2025). Check every\n  ball and ALT setting here against the S32K344EHT1MMMST package before layout. The pin table above each unit is the plan.\nSupplies: VDD_HV_A = VDD_HV_B = VREFH = 3V3_MAIN, V15 = 1V5_CORE (U303), V11/V25 internal (decoupling only).\n  NTC dividers are ratiometric to 3V3_MAIN = VREFH. Check the S32K3 supply ramp-rate limits against the LMQ66430\n  soft start (HDG 2.10.1) during bring-up.\nClock: FIRC; no FXOSC crystal in Rev A (EXTAL/XTAL no-connect; confirm the unused-pin rule in the data sheet).\nWatchdog: internal SWT, hard-locked after start-up (DEC-005). Clock monitor CMU -> reset.\nRESET_B (PTA5) on RESET_L: TPS3702 window supervisor (p3) wired-OR, PHY RESET_N, debug header pin 10.\nFlash IS25LP032D-JNLA3 on LPSPI2, mode 0 or 3, own CS with 10k pull-up so it is deselected through reset;\n  WP and HOLD pulled up (single-IO SPI). Powered from switched 3V3_MAIN; log flush before PHY sleep (DEC-007).\nDebug: Cortex 10-pin (project default). Pin 7 is the key, pin 8 unused. SWDIO 10k up, SWCLK 10k down.\nDefault states: all port pins are disabled inputs out of reset; LPSPI4 PCS0 and LPSPI2 PCS0 are held high by\n  the switch's internal pull-up and R4xx respectively; FLT and IRQ lines idle high via their pull-ups.\n"
+	(text "DESIGN NOTES (S32K3xx data sheet; S32K3 Hardware Design Guidelines Rev E2; Node60 compute page)\nRELEASE-BLOCKING (GATE-MCU-01): ball map from the library symbol (NXP IOMUX attachment, Nov 2025). Check every\n  ball and ALT setting here against the S32K344EHT1MMMST package before layout. The pin table above each unit is the plan.\nSupplies: VDD_HV_A = VDD_HV_B = VREFH = 3V3_MAIN, V15 = 1V5_CORE (U303), V11/V25 internal (decoupling only).\n  NTC dividers are ratiometric to 3V3_MAIN = VREFH. Check the S32K3 supply ramp-rate limits against the LMQ66430\n  soft start (HDG 2.10.1) during bring-up.\nClock: FIRC; no FXOSC crystal in Rev A. EXTAL/XTAL unconnected and unused GPIOs unconnected (disabled), as NXP\n  HDG Rev E2 Table 33 requires. RESET_B pulled up to VDD_HV_A (4.7k on p3), as Table 33 requires.\nWatchdog: internal SWT, hard-locked after start-up (DEC-005). Clock monitor CMU -> reset.\nRESET_B (PTA5) on RESET_L: TPS3702 window supervisor (p3) wired-OR, PHY RESET_N, debug header pin 10.\nFlash IS25LP032D-JNLA3 on LPSPI2, mode 0 or 3, own CS with 10k pull-up so it is deselected through reset;\n  WP and HOLD pulled up (single-IO SPI). Powered from switched 3V3_MAIN; log flush before PHY sleep (DEC-007).\nDebug: Cortex 10-pin (project default). Pin 7 is the key, pin 8 unused. SWDIO 10k up, SWCLK 10k down.\nDefault states: all port pins are disabled inputs out of reset; LPSPI4 PCS0 and LPSPI2 PCS0 are held high by\n  the switch's internal pull-up and R4xx respectively; FLT and IRQ lines idle high via their pull-ups.\n"
 		(exclude_from_sim no)
 		(at 236.22 368.3 0)

Commit message: DEC-015: place the ABM8AIG 16 MHz crystal on p4
- Y401 ABM8AIG-16.000MHZ-8-1Z-T on EXTAL (K1) / XTAL (L1), C424/C425
  10 pF C0G (GCM1555C1H100JA16D), R408 0R RsEXT, as NXP FRDM-A-S32K344
- Library pinned to dropout-kicad-library PR #35 head 51ade76
  (adds the three crystal candidates and the 10 pF capacitor)
- parts.yaml: selection, alternates, prices and library links;
  DEC-015 gains the start-up margin and drive-level numbers

Co-Authored-By: Claude Opus 5.5 <noreply@anthropic.com>
Parts:
- added C (x2): 10pF, DropOut_Capacitor_SMD:C_0402_1005Metric, symbol DropOut_Capacitor:GCM1555C1H100JA16D
- added R: 0R, DropOut_Resistor_SMD:R_0402_1005Metric, symbol DropOut_Resistor:AC0402JR-070RL
- added Y: ABM8AIG-16.000MHZ-8-1Z-T, DropOut_Crystal:Crystal_SMD_NDK_NX3225SA-4Pin_3.2x2.5mm, symbol DropOut_Timing:ABM8AIG-16.000MHZ-8-1Z-T
Connections:
- net GND: now also C.2, C.2, Y.2 (G), Y.4 (G)
- net FXOSC_EXTAL: now reaches U.K1 (EXTAL)
- net FXOSC_EXTAL: now also C.1, Y.1
- net FXOSC_XTAL: now reaches U.L1 (XTAL)
- net FXOSC_XTAL: now also R.1
- new net FXOSC_XTAL_X: C.1, R.2, Y.3
- no-connect marks 181 -> 179
Other:
- note added: "FXOSC (DEC-015): Y401 16 MHz, CL 8 pF, +/-10 ppm; C424/C425 10 pF C0G, R408 0R (RsEXT), as NXP FRDM-A-S32K344. gm_crit = 0.28 mA/V vs GM 9.7 mA/V min; tune C and RsEXT on the first boards (HDG E2 3.1). LAYOUT: Y401, C424, C425, R408 next to K1/L1, no vias, clean GND under them, cap grounds together (HDG E2 3.2). VREFL ties to VSS. V11 and V25 are internal regulator outputs: decoupling only, no lo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"
- note removed: "EXTAL/XTAL: no crystal in Rev A (FIRC clocks the core; RMII uses the 50 MHz oscillator). VREFL ties to VSS. V11 and V25 are internal regulator outputs: decoupling only, no loads."
