File: sheets/output-switch.kicad_sch (KiCad schematic)
At the start: 0 parts

Commit message: Schematic capture: T1S (p5) and output switch (p6-p8)
Page 5: LAN8670 with per-pin decoupling, RMII mode and PHYAD straps, the
DEC-012 line interface (C0G DC block, ACT1210E-241 choke, VETH100A1DD1
ESD, DNP 100R termination) and the 50 MHz clock feeding PHY and MCU.
Pages 6-8: one TPS2HCS08A-Q1 sheet placed three times, with the SPI
daisy chain, SNS network, VDD filter and package NTC; the root maps
each placement to OUT1..OUT6, SW1..3 and the chain nets.

Co-Authored-By: Claude Opus 5.5 <noreply@anthropic.com>
Parts:
- added C (x4): 100nF, symbol Device:C
- added C: 1uF, symbol Device:C
- added C: 470nF, symbol Device:C
- added C: 4.7nF, symbol Device:C
- added R (x4): 10k, symbol Device:R
- added R: 698R, symbol Device:R
- added R: 10R, symbol Device:R
- added R: 4.7k, symbol Device:R
- added TH: 10k, symbol Device:Thermistor_NTC
- added TP: TP_FLT_L, symbol Connector:TestPoint
- added TP: TP_SNS, symbol Connector:TestPoint
- added TP: TP_GND, symbol Connector:TestPoint
- added TP: TP_OUT_B, symbol Connector:TestPoint
- added TP: TP_OUT_A, symbol Connector:TestPoint
- added TP: TP_SDO, symbol Connector:TestPoint
- added U: TPS2HCS08AQPWPRQ1, DropOut_Package_SO:HTSSOP-16-1EP_4.4x5mm_P0.65mm_EP3.4x5mm_Mask2.78x3.313mm, symbol DropOut_PowerSwitch:TPS2HCS08AQPWPRQ1
Connections:
- new net 3V3_MAIN: R.1, R.1
- new net FLT_L: R.1, TP.1, U.12 (~{FLT}/~{WAKE_SIG})
- new net GND: C.2, C.2, C.2, C.2, C.2, C.2, C.2, R.2, R.2, R.2, TH.2, TP.1, U.1 (GND)
- new net NTC_SW: C.1, R.2, TH.1
- new net OUT_A: C.1, TP.1, U.6 (VOUT1), U.7 (VOUT1), U.8 (VOUT1)
- new net OUT_B: C.1, TP.1, U.10 (VOUT2), U.11 (VOUT2), U.9 (VOUT2)
- new net SDI: U.13 (SDI)
- new net SDO: TP.1, U.14 (SDO)
- new net SNS: R.2, TP.1
- new net SPI1_SWITCH_CS_L: U.15 (~{CS})
- new net SPI1_SWITCH_SCK: U.16 (SCLK)
- new net SW_DI: R.1, U.4 (DI)
- new net SW_LHI: R.1, U.5 (LHI)
- new net SW_SNS: C.1, R.1, R.1, U.2 (SNS)
- new net SW_VDD: C.1, R.2, R.2, U.3 (VDD)
- new net VBAT_PROT: C.1, C.1, U.17 (VBB)
Other:
- note added: "DESIGN VALUES (TPS2HCS08-Q1 SLVSHR0 sec. 9.1, Table 9-1; Node60 DEC-008, DEC-009) One file placed three times: pages 6, 7, 8 = U601 (OUT1/OUT2), U701 (OUT3/OUT4), U801 (OUT5/OUT6). SPI daisy chain (root sheet): MCU SOUT -> U601 SDI, U601 SDO -> U701 SDI, U701 SDO -> U801 SDI, U801 SDO -> MCU SIN. SCLK and CS_L shared. CRC enabled in firmware; read back every protection register (GATE-OUT-02). CSN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"
- note added: "Dual smart high-side switch, SPI daisy chain, SNS telemetry (U?01)"
- note added: "Switch VDD filter (R?01, C?03)"
- note added: "Switch-package temperature: NTC divider (R?xx, TH?01)"
- note added: "Test points"
- title: Node60 -> Node60 · E-G · Output switch (p6-p8)

Commit message: Schematic capture: MCU and NVM (p4), connectors (p9); ERC clean
Page 4: S32K344 in eight boxed units. The supply unit has decoupling per
NXP HDG Rev E2 Table 2; each port unit shows its pin plan and firmware
notes (D-14 as adopted). Pins were checked against NXP's IOMUX table:
EMAC RMII per NXP's TJA1100 use case, LPSPI4 switch chain, LPSPI2 log
flash, LPI2C0 telemetry, ADC1/ADC2 inputs, EIRQ fault lines, SWD and an
LPUART0 debug port. Also the IS25LP032D flash, the Cortex 10-pin header
and the I2C pull-ups.

Page 9: placeholder battery, return, T1S and MX150 output connectors
(all TBD selections), mirrored with pin 1 at the top (D-43), and the
PWR_FLAGs for nets entering the board.

ERC: 0 violations. 17 items are excluded in node60.kicad_pro, each with
its reason (D-52): parallel output pins typed power output in the
library (to be retyped there), and two LAN8670 pins tied to VSS per the
datasheet.

Co-Authored-By: Claude Opus 5.5 <noreply@anthropic.com>
Connections:
- net SPI1_SWITCH_CS_L renamed SPI4_SWITCH_CS_L
- net SPI1_SWITCH_SCK renamed SPI4_SWITCH_SCK
Changed lines of the file:
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@@
 		)
 	)
-	(hierarchical_label "SPI1_SWITCH_SCK"
+	(hierarchical_label "SPI4_SWITCH_SCK"
 		(shape input)
 		(at 170.18 170.18 180)
@@
 		)
 	)
-	(hierarchical_label "SPI1_SWITCH_CS_L"
+	(hierarchical_label "SPI4_SWITCH_CS_L"
 		(shape input)
 		(at 170.18 167.64 180)

Commit message: Record TBD part selections; schematic follows them
User selections of 2026-10-22: TPS7B8133QWDRVRQ1 (VDDAU LDO),
CSS2725FTL250 (0.25 mOhm RSENSE), IAUTN08S5N012LATMA1 (DGATE/HGATE
FETs, new parts entry) and NCU18XH103F6SRB (NTCs), each with its dated
DigiKey observation and the rejected or alternative candidates, which
are now parts entries too. The schematic placeholders carry the
selected MPNs until the library parts land. CCAP grows to 1uF:
10 x the summed Ciss of four IAUTN08S5N012L is 0.61 uF.

Co-Authored-By: Claude Opus 5.5 <noreply@anthropic.com>
Parts:
- TH: value 10k -> NCU18XH103F6SRB; Placeholder PLACEHOLDER: TBD part: selection pending user decision (fin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 -> PLACEHOLDER: selected 2026-10-22: Murata NCU18XH103F6SRB; l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
Changed lines of the file:
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@@
 			)
 		)
-		(property "Value" "10k"
+		(property "Value" "NCU18XH103F6SRB"
 			(at 66.548 312.42 0)
 			(effects
@@
 			)
 		)
-		(property "Placeholder" "PLACEHOLDER: TBD part: selection pending user decision (find-part), then a library session (TBD-NTC-10K: 0603, R25 1 %, B 1 %, AEC-Q200)"
+		(property "Placeholder" "PLACEHOLDER: selected 2026-10-22: Murata NCU18XH103F6SRB; library part pending (session node60-ldo-ntc)"
 			(at 63.5 311.15 0)
 			(effects

Commit message: Swap placeholders for merged DropOut library parts
Library bumped to ce98ecf (PRs #15, #16, #18, #19, #20, #21 merged).
Now real parts: IAUTN08S5N012LATMA1 (Q201-Q204, dual gate: G_ON and
G_LIN both driven), CSS2725FTL250 (R201, 2-terminal: sense nets are
VBAT_D / VBAT_Q2D with Kelvin taps from the pads in layout),
TPS7B8133QWDRVRQ1 (U301, COUT 2.2uF per its 1-200 uF requirement),
NCU18XH103F6SRB (RT201, RT601-801), Wurth 74438356022HT / 74438356010HT
buck inductors and Harwin S1751-46R GND loops (user's picks 2026-10-23),
1 mm pad test points and DT13-2P output headers. The library pin-type
fixes cut the ERC exclusions from 17 to 2. parts.yaml records the
library symbols; the library tables list the new libraries.

Co-Authored-By: Claude Opus 5.5 <noreply@anthropic.com>
Parts:
- removed TH: NCU18XH103F6SRB, symbol Device:Thermistor_NTC
- added RT: NCU18XH103F6SRB, DropOut_Resistor_SMD:R_NTC_0603_1608Metric_Pad0.7x0.7mm, symbol DropOut_Thermistor:NCU18XH103F6SRB
Connections:
- net GND: now also RT.2
- net NTC_SW: now also RT.1
Other:
- note added: "Switch-package temperature: NTC divider (R?xx, RT?01)"
- note removed: "Switch-package temperature: NTC divider (R?xx, TH?01)"
- moved on the sheet: C
Changed lines of the file:
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@@
 		)
 	)
-	(text "Switch-package temperature: NTC divider (R?xx, TH?01)"
+	(text "Switch-package temperature: NTC divider (R?xx, RT?01)"
 		(exclude_from_sim no)
 		(at 38.1 283.21 0)
@@
 	(wire
 		(pts
-			(xy 63.5 314.96)
 			(xy 63.5 317.5)
+			(xy 63.5 320.04)
 		)
 		(stroke
@@
 	(symbol
 		(lib_id "power:GND")
-		(at 63.5 317.5 0)
+		(at 63.5 320.04 0)
 		(unit 1)
 		(body_style 1)
@@
 		(dnp no)
 		(property "Reference" "#PWR015"
-			(at 63.5 317.5 0)
+			(at 63.5 320.04 0)
 			(effects
 				(font
@@
 		)
 		(property "Value" "GND"
-			(at 63.5 322.4 0)
+			(at 63.5 324.94 0)
 			(effects
 				(font
@@
 		)
 		(property "Footprint" ""
-			(at 63.5 317.5 0)
+			(at 63.5 320.04 0)
 			(effects
 				(font
@@
 		)
 		(property "Datasheet" ""
-			(at 63.5 317.5 0)
+			(at 63.5 320.04 0)
 			(effects
 				(font
@@
 	)
 	(symbol
-		(lib_id "Device:Thermistor_NTC")
-		(at 63.5 311.15 0)
+		(lib_id "DropOut_Thermistor:NCU18XH103F6SRB")
+		(at 63.5 312.42 270)
 		(unit 1)
 		(body_style 1)
@@
 		(dnp no)
 		(fields_autoplaced no)
-		(property "Reference" "TH"
-			(at 66.548 309.88 0)
-			(effects
-				(font
-					(size 1.27 1.27)
-				)
-				(justify left)
+		(property "Reference" "RT"
+			(at 67.564 311.15 270)
+			(effects
+				(font
+					(size 1.27 1.27)
+				)
+				(justify right)
 			)
 		)
 		(property "Value" "NCU18XH103F6SRB"
-			(at 66.548 312.42 0)
-			(effects
-				(font
-					(size 1.27 1.27)
-				)
-				(justify left)
-			)
-		)
-		(property "Footprint" ""
-			(at 63.5 311.15 0)
-			(effects
-				(font
-					(size 1.27 1.27)
-				)
-				(hide yes)
-			)
-		)
-		(property "Datasheet" ""
-			(at 63.5 311.15 0)
-			(effects
-				(font
-					(size 1.27 1.27)
-				)
-				(hide yes)
-			)
-		)
-		(property "Description" "Temperature dependent resistor, negative temperature coefficient"
-			(at 63.5 311.15 0)
-			(effects
-				(font
-					(size 1.27 1.27)
-				)
-				(hide yes)
-			)
-		)
-		(property "MPN" ""
-			(at 63.5 311.15 0)
-			(effects
-				(font
-					(size 1.27 1.27)
-				)
-				(hide yes)
-			)
-		)
-		(property "Manufacturer" ""
-			(at 63.5 311.15 0)
-			(effects
-				(font
-					(size 1.27 1.27)
-				)
-				(hide yes)
-			)
-		)
-		(property "DigiKey_PN" ""
-			(at 63.5 311.15 0)
-			(effects
-				(font
-					(size 1.27 1.27)
-				)
-				(hide yes)
-			)
-		)
-		(property "Mouser_PN" ""
-			(at 63.5 311.15 0)
-			(effects
-				(font
-					(size 1.27 1.27)
-				)
-				(hide yes)
-			)
-		)
-		(property "Placeholder" "PLACEHOLDER: selected 2026-10-22: Murata NCU18XH103F6SRB; library part pending (session node60-ldo-ntc)"
-			(at 63.5 311.15 0)
-			(effects
-				(font
-					(size 1.27 1.27)
-				)
-				(hide yes)
-			)
-		)
-		(property "Tolerance" "1%"
-			(at 63.5 311.15 0)
+			(at 67.564 313.69 270)
+			(effects
+				(font
+					(size 1.27 1.27)
+				)
+				(justify right)
+			)
+		)
+		(property "Footprint" "DropOut_Resistor_SMD:R_NTC_0603_1608Metric_Pad0.7x0.7mm"
+			(at 63.5 312.42 0)
+			(effects
+				(font
+					(size 1.27 1.27)
+				)
+				(hide yes)
+			)
+		)
+		(property "Datasheet" "https://www.murata.com/en-us/products/productdetail?partno=NCU18XH103F6SRB"
+			(at 63.5 312.42 0)
+			(effects
+				(font
+					(size 1.27 1.27)
+				)
+				(hide yes)
+			)
+		)
+		(property "Description" "Murata NCU18 NTC thermistor 10 kΩ ±1 %, B25/50 3380 K ±1 %, -55 to +150 °C, automotive (AEC-Q200), 0603 (1608 metric)"
+			(at 63.5 312.42 0)
+			(effects
+				(font
+					(size 1.27 1.27)
+				)
+				(hide yes)
+			)
+		)
+		(property "Manufacturer" "Murata Electronics"
+			(at 63.5 312.42 0)
+			(effects
+				(font
+					(size 1.27 1.27)
+				)
+				(hide yes)
+			)
+		)
+		(property "MPN" "NCU18XH103F6SRB"
+			(at 63.5 312.42 0)
+			(effects
+				(font
+					(size 1.27 1.27)
+				)
+				(hide yes)
+			)
+		)
+		(property "DigiKey_PN" "490-18139-1-ND"
+			(at 63.5 312.42 0)
+			(effects
+				(font
+					(size 1.27 1.27)
+				)
+				(hide yes)
+			)
+		)
+		(property "Mouser_PN" "81-NCU18XH103F6SRB"
+			(at 63.5 312.42 0)
+			(effects
+				(font
+					(size 1.27 1.27)
+				)
+				(hide yes)
+			)
+		)
+		(property "Temperature_Grade" "AEC-Q200, -55 to +150 °C"
+			(at 63.5 312.42 0)
+			(effects
+				(font
+					(size 1.27 1.27)
+				)
+				(hide yes)
+			)
+		)
+		(property "Notes" "R-T table on Murata's product page (Resistance-Temperature Characteristics); XH103 centre values in catalog R44E p. 15"
+			(at 63.5 312.42 0)
 			(effects
 				(font
@@
 			(project "node60"
 				(path "/55f51841-30a3-4965-b848-b796f60054d0/ceecbbf6-496b-4919-aa4d-b8194f44838e"
-					(reference "TH601")
+					(reference "RT601")
 					(unit 1)
 				)
 				(path "/55f51841-30a3-4965-b848-b796f60054d0/68ca6db2-fb88-4c17-b54b-7131815c5345"
-					(reference "TH701")
+					(reference "RT701")
 					(unit 1)
 				)
 				(path "/55f51841-30a3-4965-b848-b796f60054d0/618ad5c3-1fe8-46d2-96b6-b9e1aa40313d"
-					(reference "TH801")
+					(reference "RT801")
 					(unit 1)
 				)
@@
 		(pts
 			(xy 63.5 307.34)
-			(xy 96.52 307.34)
+			(xy 101.6 307.34)
 		)
 		(stroke
@@
 	(wire
 		(pts
-			(xy 76.2 307.34)
-			(xy 76.2 309.88)
+			(xy 88.9 307.34)
+			(xy 88.9 309.88)
 		)
 		(stroke
@@
 	(wire
 		(pts
-			(xy 76.2 317.5)
-			(xy 76.2 320.04)
+			(xy 88.9 317.5)
+			(xy 88.9 320.04)
 		)
 		(stroke
@@
 	(symbol
 		(lib_id "power:GND")
-		(at 76.2 320.04 0)
+		(at 88.9 320.04 0)
 		(unit 1)
 		(body_style 1)
@@
 		(dnp no)
 		(property "Reference" "#PWR016"
-			(at 76.2 320.04 0)
+			(at 88.9 320.04 0)
 			(effects
 				(font
@@
 		)
 		(property "Value" "GND"
-			(at 76.2 324.94 0)
+			(at 88.9 324.94 0)
 			(effects
 				(font
@@
 		)
 		(property "Footprint" ""
-			(at 76.2 320.04 0)
+			(at 88.9 320.04 0)
 			(effects
 				(font
@@
 		)
 		(property "Datasheet" ""
-			(at 76.2 320.04 0)
+			(at 88.9 320.04 0)
 			(effects
 				(font
@@
 	(symbol
 		(lib_id "Device:C")
-		(at 76.2 313.69 0)
+		(at 88.9 313.69 0)
 		(unit 1)
 		(body_style 1)
@@
 		(fields_autoplaced no)
 		(property "Reference" "C"
-			(at 79.502 312.42 0)
+			(at 92.202 312.42 0)
 			(effects
 				(font
@@
 		)
 		(property "Value" "100nF"
-			(at 79.502 314.96 0)
+			(at 92.202 314.96 0)
 			(effects
 				(font
@@
 		)
 		(property "Footprint" ""
-			(at 76.2 313.69 0)
+			(at 88.9 313.69 0)
 			(effects
 				(font
@@
 		)
 		(property "Datasheet" ""
-			(at 76.2 313.69 0)
+			(at 88.9 313.69 0)
 			(effects
 				(font
@@
 		)
 		(property "Description" "Unpolarized capacitor"
-			(at 76.2 313.69 0)
+			(at 88.9 313.69 0)
 			(effects
 				(font
@@
 		)
 		(property "MPN" ""
-			(at 76.2 313.69 0)
+			(at 88.9 313.69 0)
 			(effects
 				(font
@@
 		)
 		(property "Manufacturer" ""
-			(at 76.2 313.69 0)
+			(at 88.9 313.69 0)
 			(effects
 				(font
@@
 		)
 		(property "DigiKey_PN" ""
-			(at 76.2 313.69 0)
+			(at 88.9 313.69 0)
 			(effects
 				(font
@@
 		)
 		(property "Mouser_PN" ""
-			(at 76.2 313.69 0)
+			(at 88.9 313.69 0)
 			(effects
 				(font
@@
 		)
 		(property "Placeholder" "PLACEHOLDER: awaiting DropOut_Resistor/DropOut_Capacitor part (library brief 01-passives)"
-			(at 76.2 313.69 0)
+			(at 88.9 313.69 0)
 			(effects
 				(font
@@
 		)
 		(property "Voltage" "25V"
-			(at 76.2 313.69 0)
+			(at 88.9 313.69 0)
 			(effects
 				(font
@@
 		)
 		(property "Dielectric" "C0G"
-			(at 76.2 313.69 0)
+			(at 88.9 313.69 0)
 			(effects
 				(font
@@
 		)
 		(property "Package" "0805"
-			(at 76.2 313.69 0)
+			(at 88.9 313.69 0)
 			(effects
 				(font
@@
 		)
 		(property "Tolerance" "5%"
-			(at 76.2 313.69 0)
+			(at 88.9 313.69 0)
 			(effects
 				(font
@@
 	(hierarchical_label "NTC_SW"
 		(shape output)
-		(at 96.52 307.34 0)
+		(at 101.6 307.34 0)
 		(effects
 			(font
@@
 	)
 	(junction
-		(at 76.2 307.34)
+		(at 88.9 307.34)
 		(diameter 0)
 		(color 0 0 0 0)

Commit message: Swap all resistors, capacitors and test points for DropOut parts
Library bumped to 752b63c (PR #22: 83 AEC-Q200 chip resistors and MLCCs,
PR #24: passive symbol layout). Each passive is now a real part, chosen
by rule: exact value and dielectric, tolerance and voltage at least as
good, the drawn package else the next larger, then manufacturer order;
the other built sources stay in the library as alternates.

Where the library has no part in the drawn package: 10nF C0G, 4.7nF C0G,
1uF 16V and 470nF 16V 0402 -> 0603; 68nF C0G, 100nF C0G and 10uF 16V
0805 -> 1206; 32k 1% -> 0.1% (TNPW060332K0BEEA); CCAP 1uF 50V (not built)
-> 1uF 100V 1206. 0R debug links on regulator outputs use the 5 A
CRCW06030000Z0EAHP jumper.

Also fixes test points: f9af1d2 described them as swapped, but they were
still stock symbols. They are now TestPoint_Pad_D1.0mm (signals) and
Harwin S1751-46R (GND loops).

Only placeholders left: L201 / C208 (EMI filter, TBD) and J901-J903.

Co-Authored-By: Claude Opus 5.5 <noreply@anthropic.com>
Parts:
- C: footprint (none) -> DropOut_Capacitor_SMD:C_0603_1608Metric; symbol Device:C -> DropOut_Capacitor:GCJ188R72A104KA01D; Case (none) -> 0603; DigiKey_PN (none) -> 490-13420-1-ND; MPN (none) -> GCJ188R72A104KA01D; Manufacturer (none) -> Murata; Mouser_PN (none) -> 81-GCJ188R72A104KA1D; Notes (none) -> Murata makes no 100 V 100 nF X7R GCM in 0603; GCJ is Murata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; Package 0603 -> (none); Placeholder PLACEHOLDER: awaiting DropOut_Resistor/DropOut_Capacitor pa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 -> (none); Temperature_Grade (none) -> AEC-Q200, -55 to +125 °C; Tolerance 10% -> ±10%
- C: footprint (none) -> DropOut_Capacitor_SMD:C_1206_3216Metric; symbol Device:C -> DropOut_Capacitor:GCM31C5C2A104JE02L; Case (none) -> 1206; DigiKey_PN (none) -> 490-GCM31C5C2A104JE02LCT-ND; MPN (none) -> GCM31C5C2A104JE02L; Manufacturer (none) -> Murata; Mouser_PN (none) -> 81-GCM31C5C2A104JE2L; Package 0805 -> (none); Placeholder PLACEHOLDER: awaiting DropOut_Resistor/DropOut_Capacitor pa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 -> (none); Temperature_Grade (none) -> AEC-Q200, -55 to +125 °C; Tolerance 5% -> ±5%; Voltage 25V -> 100V
- C: footprint (none) -> DropOut_Capacitor_SMD:C_1206_3216Metric; symbol Device:C -> DropOut_Capacitor:CGA5L2X7R2A105K160AA; Case (none) -> 1206; DigiKey_PN (none) -> 445-5845-1-ND; MPN (none) -> CGA5L2X7R2A105K160AA; Manufacturer (none) -> TDK; Mouser_PN (none) -> 810-CGA5L2X7R2A105K; Package 1206 -> (none); Placeholder PLACEHOLDER: awaiting DropOut_Resistor/DropOut_Capacitor pa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 -> (none); Temperature_Grade (none) -> AEC-Q200, -55 to +125 °C; Tolerance 10% -> ±10%
- C: footprint (none) -> DropOut_Capacitor_SMD:C_0603_1608Metric; symbol Device:C -> DropOut_Capacitor:GCM188R71C474KA55D; Case (none) -> 0603; DigiKey_PN (none) -> 490-4775-1-ND; MPN (none) -> GCM188R71C474KA55D; Manufacturer (none) -> Murata; Mouser_PN (none) -> 81-GCM188R71C474KA5D; Notes (none) -> No AEC-Q200 part exists in the drawn 0402 package (DigiKey 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; Package 0402 -> (none); Placeholder PLACEHOLDER: awaiting DropOut_Resistor/DropOut_Capacitor pa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 -> (none); Temperature_Grade (none) -> AEC-Q200, -55 to +125 °C; Tolerance 10% -> ±10%
- C: footprint (none) -> DropOut_Capacitor_SMD:C_0603_1608Metric; symbol Device:C -> DropOut_Capacitor:GCM1885C1H472JA16D; Case (none) -> 0603; DigiKey_PN (none) -> 490-GCM1885C1H472JA16DCT-ND; MPN (none) -> GCM1885C1H472JA16D; Manufacturer (none) -> Murata; Mouser_PN (none) -> 81-GCM1885C1H472JA6D; Notes (none) -> No AEC-Q200 part exists in the drawn 0402 package (DigiKey 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; Package 0402 -> (none); Placeholder PLACEHOLDER: awaiting DropOut_Resistor/DropOut_Capacitor pa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 -> (none); Temperature_Grade (none) -> AEC-Q200, -55 to +125 °C; Tolerance 5% -> ±5%
- R: footprint (none) -> DropOut_Resistor_SMD:R_0402_1005Metric; symbol Device:R -> DropOut_Resistor:AC0402JR-0710KL; Case (none) -> 0402; DigiKey_PN (none) -> YAG3517CT-ND; MPN (none) -> AC0402JR-0710KL; Manufacturer (none) -> Yageo; Mouser_PN (none) -> 603-AC0402JR-0710KL; Package 0402 -> (none); Placeholder PLACEHOLDER: awaiting DropOut_Resistor/DropOut_Capacitor pa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 -> (none); Power (none) -> 1/16W; Temperature_Grade (none) -> AEC-Q200, -55 to +155 °C; Tolerance 5% -> ±5%; Voltage (none) -> 50V
- R: footprint (none) -> DropOut_Resistor_SMD:R_0603_1608Metric; symbol Device:R -> DropOut_Resistor:ERA-3AEB6980V; Case (none) -> 0603; DigiKey_PN (none) -> 10-ERA-3AEB6980VCT-ND; MPN (none) -> ERA-3AEB6980V; Manufacturer (none) -> Panasonic; Mouser_PN (none) -> 667-ERA-3AEB6980V; Notes (none) -> Precision part: not substitutable (0.1 %, ±25 ppm/K thin fi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; Package 0603 -> (none); Placeholder PLACEHOLDER: awaiting DropOut_Resistor/DropOut_Capacitor pa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 -> (none); Power (none) -> 0.1W; Tempco 25ppm -> (none); Temperature_Grade (none) -> AEC-Q200, -55 to +155 °C; Tolerance 0.1% -> ±0.1%; Voltage (none) -> 75V
- R: footprint (none) -> DropOut_Resistor_SMD:R_0603_1608Metric; symbol Device:R -> DropOut_Resistor:ERA-3AEB103V; Case (none) -> 0603; DigiKey_PN (none) -> P10KDBCT-ND; MPN (none) -> ERA-3AEB103V; Manufacturer (none) -> Panasonic; Mouser_PN (none) -> 667-ERA-3AEB103V; Notes (none) -> Precision part: not substitutable (0.1 %, ±25 ppm/K thin fi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; Package 0603 -> (none); Placeholder PLACEHOLDER: awaiting DropOut_Resistor/DropOut_Capacitor pa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 -> (none); Power (none) -> 0.1W; Tempco 25ppm -> (none); Temperature_Grade (none) -> AEC-Q200, -55 to +155 °C; Tolerance 0.1% -> ±0.1%; Voltage (none) -> 75V
- R: footprint (none) -> DropOut_Resistor_SMD:R_0402_1005Metric; symbol Device:R -> DropOut_Resistor:AC0402JR-0710RL; Case (none) -> 0402; DigiKey_PN (none) -> YAG3519CT-ND; MPN (none) -> AC0402JR-0710RL; Manufacturer (none) -> Yageo; Mouser_PN (none) -> 603-AC0402JR-0710RL; Package 0402 -> (none); Placeholder PLACEHOLDER: awaiting DropOut_Resistor/DropOut_Capacitor pa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 -> (none); Power (none) -> 1/16W; Temperature_Grade (none) -> AEC-Q200, -55 to +155 °C; Tolerance 5% -> ±5%; Voltage (none) -> 50V
- R: footprint (none) -> DropOut_Resistor_SMD:R_0402_1005Metric; symbol Device:R -> DropOut_Resistor:AC0402JR-074K7L; Case (none) -> 0402; DigiKey_PN (none) -> 311-4.7KLBCT-ND; MPN (none) -> AC0402JR-074K7L; Manufacturer (none) -> Yageo; Mouser_PN (none) -> 603-AC0402JR-074K7L; Package 0402 -> (none); Placeholder PLACEHOLDER: awaiting DropOut_Resistor/DropOut_Capacitor pa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 -> (none); Power (none) -> 1/16W; Temperature_Grade (none) -> AEC-Q200, -55 to +155 °C; Tolerance 5% -> ±5%; Voltage (none) -> 50V
- TP: value TP_FLT_L -> TestPoint_Pad_D1.0mm; footprint (none) -> DropOut_TestPoint:TestPoint_Pad_D1.0mm; symbol Connector:TestPoint -> DropOut_Connector:TestPoint_Pad_D1.0mm; DigiKey_PN (none) -> -; MPN (none) -> TestPoint_Pad_D1.0mm; Manufacturer (none) -> DropOut; Mouser_PN (none) -> -; Notes (none) -> PCB copper only; nothing to order. Excluded from BOM and po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; Placeholder PLACEHOLDER: awaiting DropOut test-point part (library brie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 -> (none); Type 1mm pad -> (none)
- TP: value TP_SNS -> TestPoint_Pad_D1.0mm; footprint (none) -> DropOut_TestPoint:TestPoint_Pad_D1.0mm; symbol Connector:TestPoint -> DropOut_Connector:TestPoint_Pad_D1.0mm; DigiKey_PN (none) -> -; MPN (none) -> TestPoint_Pad_D1.0mm; Manufacturer (none) -> DropOut; Mouser_PN (none) -> -; Notes (none) -> PCB copper only; nothing to order. Excluded from BOM and po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; Placeholder PLACEHOLDER: awaiting DropOut test-point part (library brie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 -> (none); Type 1mm pad -> (none)
- TP: value TP_GND -> S1751-46R; footprint (none) -> DropOut_TestPoint:TestPoint_Harwin_S1751; symbol Connector:TestPoint -> DropOut_Connector:S1751-46R; DigiKey_PN (none) -> 952-1478-1-ND; MPN (none) -> S1751-46R; Manufacturer (none) -> Harwin; Mouser_PN (none) -> 855-S1751-46R; Notes (none) -> Ground test point (probe loop) for a scope ground spring or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; Placeholder PLACEHOLDER: awaiting DropOut test-point part (library brie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 -> (none); Temperature_Grade (none) -> -55 to +125 °C; Type probe loop -> (none)
- TP: value TP_OUT_B -> TestPoint_Pad_D1.0mm; footprint (none) -> DropOut_TestPoint:TestPoint_Pad_D1.0mm; symbol Connector:TestPoint -> DropOut_Connector:TestPoint_Pad_D1.0mm; DigiKey_PN (none) -> -; MPN (none) -> TestPoint_Pad_D1.0mm; Manufacturer (none) -> DropOut; Mouser_PN (none) -> -; Notes (none) -> PCB copper only; nothing to order. Excluded from BOM and po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; Placeholder PLACEHOLDER: awaiting DropOut test-point part (library brie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 -> (none); Type 1mm pad -> (none)
- TP: value TP_OUT_A -> TestPoint_Pad_D1.0mm; footprint (none) -> DropOut_TestPoint:TestPoint_Pad_D1.0mm; symbol Connector:TestPoint -> DropOut_Connector:TestPoint_Pad_D1.0mm; DigiKey_PN (none) -> -; MPN (none) -> TestPoint_Pad_D1.0mm; Manufacturer (none) -> DropOut; Mouser_PN (none) -> -; Notes (none) -> PCB copper only; nothing to order. Excluded from BOM and po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; Placeholder PLACEHOLDER: awaiting DropOut test-point part (library brie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 -> (none); Type 1mm pad -> (none)
- TP: value TP_SDO -> TestPoint_Pad_D1.0mm; footprint (none) -> DropOut_TestPoint:TestPoint_Pad_D1.0mm; symbol Connector:TestPoint -> DropOut_Connector:TestPoint_Pad_D1.0mm; DigiKey_PN (none) -> -; MPN (none) -> TestPoint_Pad_D1.0mm; Manufacturer (none) -> DropOut; Mouser_PN (none) -> -; Notes (none) -> PCB copper only; nothing to order. Excluded from BOM and po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; Placeholder PLACEHOLDER: awaiting DropOut test-point part (library brie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 -> (none); Type 1mm pad -> (none)
