File: sheets/output-switch.kicad_sch (KiCad schematic)
At the start: 22 parts

Commit message: Schematic: LHI to the MCU, current notes, net-name map
- LHI on all three TPS2HCS08 is now SW_LHI from S32K344 PTE4 (the
  architecture's GPIO list), still held low by the 10k pull-downs
  through reset.
- Page 4 cites NXP HDG Rev E2 Table 33 for unused GPIO, EXTAL/XTAL and
  the RESET_B pull-up instead of an open 'confirm' note.
- Copper notes for the 10 A output paths (p6) and the 60 A path (p2,
  p9), as IPC-2221 starting estimates to confirm with IPC-2152.
- interfaces.mdx maps the architecture's signal names to the schematic
  nets (RESET_L, T1S_IRQ_L, *_FLT_L, SPI4/SPI2/I2C0 buses).

Co-Authored-By: Claude Opus 5.5 <noreply@anthropic.com>
Changed lines of the file:
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@@
 		)
 	)
-	(label "SW_LHI"
+	(hierarchical_label "SW_LHI"
+		(shape input)
 		(at 144.78 162.56 0)
 		(effects
@@
 				(size 1.27 1.27)
 			)
-			(justify left bottom)
+			(justify left)
 		)
 	)
@@
 		)
 	)
-	(text "DESIGN VALUES (TPS2HCS08-Q1 SLVSHR0 sec. 9.1, Table 9-1; Node60 DEC-008, DEC-009)\nOne file placed three times: pages 6, 7, 8 = U601 (OUT1/OUT2), U701 (OUT3/OUT4), U801 (OUT5/OUT6).\nSPI daisy chain (root sheet): MCU SOUT -> U601 SDI, U601 SDO -> U701 SDI, U701 SDO -> U801 SDI, U801 SDO -> MCU SIN.\n  SCLK and CS_L shared. CRC enabled in firmware; read back every protection register (GATE-OUT-02).\n  CSN and SDO are pulled up internally to VDD; CSN idles high, so all channels stay off after reset.\nVDD: 3V3_MAIN through RVDD 10R (limits VDD slew), CVDD 470nF at the pin (TI Table 9-1). Same 3.3 V as the MCU I/O.\nVBB (exposed pad) on VBAT_PROT, CVBB2 1uF + 100nF 100 V. Broad copper and a via array under the pad.\nDI and LHI held low through 10k (TI: DI needs 10k protection): limp-home not used, LHI hardware-inactive.\nFLT/WAKE_SIG open drain, 4.7k pull-up to the VDD pin (TI Table 9-1) -> one fault line per device to the MCU.\nSNS: RSNS 698R 0.1 % 25 ppm || CSNS 4.7nF C0G at the pin (TI: 0.2-1.5k, 1-4.7nF), RPROT 10k to the MCU ADC.\n  KSNS1 = 5000: 10 A -> 2 mA x 698R = 1.396 V; 100 mA -> 13.96 mV = 17.3 counts (3.3 V / 4096).\n  The SPI-selected channel is stored with every sample. Rev A keeps KSNS1 while I2t is active (DEC-009).\nCOUT 100nF 100 V per channel (TI: 22-100nF; 100nF for hot short in MANUAL_LPM).\nEach output path: 10 A target, 14 AWG minimum; 8 A/ch is the datasheet limit with both channels on at 85 C.\nRELEASE BLOCKER: 10 A continuous unproven until GATE-THM-01 passes (dual-channel thermal test).\nPackage NTC: 10k 0.1 % over NTC to GND, 100nF C0G; place beside U?01 (GATE-TMP-01).\n"
+	(text "DESIGN VALUES (TPS2HCS08-Q1 SLVSHR0 sec. 9.1, Table 9-1; Node60 DEC-008, DEC-009)\nOne file placed three times: pages 6, 7, 8 = U601 (OUT1/OUT2), U701 (OUT3/OUT4), U801 (OUT5/OUT6).\nSPI daisy chain (root sheet): MCU SOUT -> U601 SDI, U601 SDO -> U701 SDI, U701 SDO -> U801 SDI, U801 SDO -> MCU SIN.\n  SCLK and CS_L shared. CRC enabled in firmware; read back every protection register (GATE-OUT-02).\n  CSN and SDO are pulled up internally to VDD; CSN idles high, so all channels stay off after reset.\nVDD: 3V3_MAIN through RVDD 10R (limits VDD slew), CVDD 470nF at the pin (TI Table 9-1). Same 3.3 V as the MCU I/O.\nVBB (exposed pad) on VBAT_PROT, CVBB2 1uF + 100nF 100 V. Broad copper and a via array under the pad.\nDI held low through 10k (TI: DI needs 10k protection). LHI (limp home, active high) comes from MCU PTE4 as SW_LHI,\n  shared by all three switches, with a 10k pull-down per device (3.3k total): inactive through reset and while the\n  MCU is unpowered; firmware never asserts it in normal operation.\nCURRENT (layout): OUT_A / OUT_B carry 10 A each. IPC-2221 external-layer estimate for 20 C rise: about 2.3 mm on\n  2 oz copper (256 mil2); use pours on several layers and >= 10 x 0.3 mm vias per layer change, then check with\n  IPC-2152 at +125 C ambient. Each DT13-2P pin 2 return is sized the same.\nFLT/WAKE_SIG open drain, 4.7k pull-up to the VDD pin (TI Table 9-1) -> one fault line per device to the MCU.\nSNS: RSNS 698R 0.1 % 25 ppm || CSNS 4.7nF C0G at the pin (TI: 0.2-1.5k, 1-4.7nF), RPROT 10k to the MCU ADC.\n  KSNS1 = 5000: 10 A -> 2 mA x 698R = 1.396 V; 100 mA -> 13.96 mV = 17.3 counts (3.3 V / 4096).\n  The SPI-selected channel is stored with every sample. Rev A keeps KSNS1 while I2t is active (DEC-009).\nCOUT 100nF 100 V per channel (TI: 22-100nF; 100nF for hot short in MANUAL_LPM).\nEach output path: 10 A target, 14 AWG minimum; 8 A/ch is the datasheet limit with both channels on at 85 C.\nRELEASE BLOCKER: 10 A continuous unproven until GATE-THM-01 passes (dual-channel thermal test).\nPackage NTC: 10k 0.1 % over NTC to GND, 100nF C0G; place beside U?01 (GATE-TMP-01).\n"
 		(exclude_from_sim no)
 		(at 304.8 40.64 0)

Commit message: Pin DropOut library to main 618de03 (PR #35 merged)
The re-pin also brings library PRs #31, #33 and #34 (manufacturer names,
ATM13 Notes, catalog data). Their field changes are copied into the
schematic so every placed symbol matches the library: "Amphenol Sine
Systems", "Stackpole Electronics", "Murata", and the full ATM13 Notes.

Co-Authored-By: Claude Opus 5.5 <noreply@anthropic.com>
Parts:
- RT: Manufacturer Murata Electronics -> Murata
Changed lines of the file:
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@@
 			)
 		)
-		(property "Manufacturer" "Murata Electronics"
+		(property "Manufacturer" "Murata"
 			(at 63.5 312.42 0)
 			(effects

Commit message: One LPSPI bus per output switch (DEC-018); Zephyr as core RTOS (DEC-019)
- Split the TPS2HCS08A daisy chain into three buses: U601 on LPSPI4 (Rev A
  balls), U701 on LPSPI5 (A16/A15/B13/G16), U801 on LPSPI3 (E14/F14/E15/G15).
  The output-switch sheet now exposes generic SDI/SDO/SCK/CS_L ports.
- Per-switch SPI watchdog (400 ms) with limp-home off: a lost bus turns only
  that switch's two outputs off.
- DEC-019 records Zephyr with a driver map; pin plan reviewed against
  upstream Zephyr (EIRQ map, ADC group-channel, native PCS). No other pin moves.
- GATE-MCU-01 reopened for the eight new balls (IBIS/BSDL machine check done,
  user sign-off pending). Rev B (in progress) listed on the revisions page.

Co-Authored-By: Claude Opus 5.5 <noreply@anthropic.com>
Connections:
- net SPI4_SWITCH_CS_L renamed CS_L
- net SPI4_SWITCH_SCK renamed SCK
Other:
- note added: "DESIGN VALUES (TPS2HCS08-Q1 SLVSHR0 sec. 9.1, Table 9-1; Node60 DEC-008, DEC-009) One file placed three times: pages 6, 7, 8 = U601 (OUT1/OUT2), U701 (OUT3/OUT4), U801 (OUT5/OUT6). SPI (root sheet, DEC-018): one MCU LPSPI bus per switch, SDI/SDO/SCK/CS_L not shared: U601 = LPSPI4, U701 = LPSPI5, U801 = LPSPI3. Mode 1, 8 MHz max. CRC and SPI watchdog enabled in firmware; read back every protection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"
- note added: "Dual smart high-side switch, own SPI bus, SNS telemetry (U?01)"
- note removed: "DESIGN VALUES (TPS2HCS08-Q1 SLVSHR0 sec. 9.1, Table 9-1; Node60 DEC-008, DEC-009) One file placed three times: pages 6, 7, 8 = U601 (OUT1/OUT2), U701 (OUT3/OUT4), U801 (OUT5/OUT6). SPI daisy chain (root sheet): MCU SOUT -> U601 SDI, U601 SDO -> U701 SDI, U701 SDO -> U801 SDI, U801 SDO -> MCU SIN. SCLK and CS_L shared. CRC enabled in firmware; read back every protection register (GATE-OUT-02). CSN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"
- note removed: "Dual smart high-side switch, SPI daisy chain, SNS telemetry (U?01)"
Changed lines of the file:
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@@
 		)
 	)
-	(text "Dual smart high-side switch, SPI daisy chain, SNS telemetry (U?01)"
+	(text "Dual smart high-side switch, own SPI bus, SNS telemetry (U?01)"
 		(exclude_from_sim no)
 		(at 83.82 87.63 0)
@@
 		)
 	)
-	(hierarchical_label "SPI4_SWITCH_SCK"
+	(hierarchical_label "SCK"
 		(shape input)
 		(at 170.18 170.18 180)
@@
 		)
 	)
-	(hierarchical_label "SPI4_SWITCH_CS_L"
+	(hierarchical_label "CS_L"
 		(shape input)
 		(at 170.18 167.64 180)
@@
 		)
 	)
-	(text "DESIGN VALUES (TPS2HCS08-Q1 SLVSHR0 sec. 9.1, Table 9-1; Node60 DEC-008, DEC-009)\nOne file placed three times: pages 6, 7, 8 = U601 (OUT1/OUT2), U701 (OUT3/OUT4), U801 (OUT5/OUT6).\nSPI daisy chain (root sheet): MCU SOUT -> U601 SDI, U601 SDO -> U701 SDI, U701 SDO -> U801 SDI, U801 SDO -> MCU SIN.\n  SCLK and CS_L shared. CRC enabled in firmware; read back every protection register (GATE-OUT-02).\n  CSN and SDO are pulled up internally to VDD; CSN idles high, so all channels stay off after reset.\nVDD: 3V3_MAIN through RVDD 10R (limits VDD slew), CVDD 470nF at the pin (TI Table 9-1). Same 3.3 V as the MCU I/O.\nVBB (exposed pad) on VBAT_PROT, CVBB2 1uF + 100nF 100 V. Broad copper and a via array under the pad.\nDI held low through 10k (TI: DI needs 10k protection). LHI (limp home, active high) comes from MCU PTE4 as SW_LHI,\n  shared by all three switches, with a 10k pull-down per device (3.3k total): inactive through reset and while the\n  MCU is unpowered; firmware never asserts it in normal operation.\nCURRENT (layout): OUT_A / OUT_B carry 10 A each. IPC-2221 external-layer estimate for 20 C rise: about 2.3 mm on\n  2 oz copper (256 mil2); use pours on several layers and >= 10 x 0.3 mm vias per layer change, then check with\n  IPC-2152 at +125 C ambient. Each DT13-2P pin 2 return is sized the same.\nFLT/WAKE_SIG open drain, 4.7k pull-up to the VDD pin (TI Table 9-1) -> one fault line per device to the MCU.\nSNS: RSNS 698R 0.1 % 25 ppm || CSNS 4.7nF C0G at the pin (TI: 0.2-1.5k, 1-4.7nF), RPROT 10k to the MCU ADC.\n  KSNS1 = 5000: 10 A -> 2 mA x 698R = 1.396 V; 100 mA -> 13.96 mV = 17.3 counts (3.3 V / 4096).\n  The SPI-selected channel is stored with every sample. Rev A keeps KSNS1 while I2t is active (DEC-009).\nCOUT 100nF 100 V per channel (TI: 22-100nF; 100nF for hot short in MANUAL_LPM).\nEach output path: 10 A target, 14 AWG minimum; 8 A/ch is the datasheet limit with both channels on at 85 C.\nRELEASE BLOCKER: 10 A continuous unproven until GATE-THM-01 passes (dual-channel thermal test).\nPackage NTC: 10k 0.1 % over NTC to GND, 100nF C0G; place beside U?01 (GATE-TMP-01).\n"
+	(text "DESIGN VALUES (TPS2HCS08-Q1 SLVSHR0 sec. 9.1, Table 9-1; Node60 DEC-008, DEC-009)\nOne file placed three times: pages 6, 7, 8 = U601 (OUT1/OUT2), U701 (OUT3/OUT4), U801 (OUT5/OUT6).\nSPI (root sheet, DEC-018): one MCU LPSPI bus per switch, SDI/SDO/SCK/CS_L not shared: U601 = LPSPI4, U701 = LPSPI5,\n  U801 = LPSPI3. Mode 1, 8 MHz max. CRC and SPI watchdog enabled in firmware; read back every protection register (GATE-OUT-02).\n  CSN and SDO are pulled up internally to VDD; CSN idles high, so all channels stay off after reset.\nVDD: 3V3_MAIN through RVDD 10R (limits VDD slew), CVDD 470nF at the pin (TI Table 9-1). Same 3.3 V as the MCU I/O.\nVBB (exposed pad) on VBAT_PROT, CVBB2 1uF + 100nF 100 V. Broad copper and a via array under the pad.\nDI held low through 10k (TI: DI needs 10k protection). LHI (limp home, active high) comes from MCU PTE4 as SW_LHI,\n  shared by all three switches, with a 10k pull-down per device (3.3k total): inactive through reset and while the\n  MCU is unpowered; firmware never asserts it in normal operation.\nCURRENT (layout): OUT_A / OUT_B carry 10 A each. IPC-2221 external-layer estimate for 20 C rise: about 2.3 mm on\n  2 oz copper (256 mil2); use pours on several layers and >= 10 x 0.3 mm vias per layer change, then check with\n  IPC-2152 at +125 C ambient. Each DT13-2P pin 2 return is sized the same.\nFLT/WAKE_SIG open drain, 4.7k pull-up to the VDD pin (TI Table 9-1) -> one fault line per device to the MCU.\nSNS: RSNS 698R 0.1 % 25 ppm || CSNS 4.7nF C0G at the pin (TI: 0.2-1.5k, 1-4.7nF), RPROT 10k to the MCU ADC.\n  KSNS1 = 5000: 10 A -> 2 mA x 698R = 1.396 V; 100 mA -> 13.96 mV = 17.3 counts (3.3 V / 4096).\n  The SPI-selected channel is stored with every sample. Rev A keeps KSNS1 while I2t is active (DEC-009).\nCOUT 100nF 100 V per channel (TI: 22-100nF; 100nF for hot short in MANUAL_LPM).\nEach output path: 10 A target, 14 AWG minimum; 8 A/ch is the datasheet limit with both channels on at 85 C.\nRELEASE BLOCKER: 10 A continuous unproven until GATE-THM-01 passes (dual-channel thermal test).\nPackage NTC: 10k 0.1 % over NTC to GND, 100nF C0G; place beside U?01 (GATE-TMP-01).\n"
 		(exclude_from_sim no)
 		(at 304.8 40.64 0)
